File: Hardware/board/board.kicad_pcb (KiCad board)
At the start: 2 copper layers, 49 parts, among them J1 USB_C_Receptacle_USB2.0_16P, J2 Barrel_Jack_PTH, SW1 SKRPACE010, SW10 CPG151101D212, SW11 CPG151101D212, SW12 CPG151101D212, SW13 CPG151101D212, SW14 CPG151101D212, SW15 CPG151101D212, SW2 EC11E15244G1, SW3 EC11E15244G1, SW4 EC11E15244G1, SW5 EC11E15244G1, SW6 EC11E15244G1, SW7 EC11E15244G1, SW8 CPG151101D212, SW9 CPG151101D212, U1 MIC5219-3.3YM5, U2 MIC5219-3.3YM5, U3 STM32F407VETx, U4 HC-FPC-0.5-40P-FH20, U5 PT4103B23F, X1 CSTNE8M00G550000R0

Commit message: desigin designing
dsa
Parts:
- added C18: 100nF, PCM_fab:C_0603, F.Cu at (204.7, 76.9)
- added C19: 22uF, Capacitor_SMD:C_0805_2012Metric, F.Cu at (199.6, 155.7)
- added C20: 22uF, PCM_fab:C_0603, F.Cu at (186.7, 164.5)
- added C21: 22uF, Capacitor_SMD:C_0805_2012Metric, F.Cu at (195.2, 155.7)
- added C22: 22uF, PCM_fab:C_0603, F.Cu at (186.7, 159.5)
- added C23: 22uF, Capacitor_SMD:C_0805_2012Metric, F.Cu at (195.2, 158.7)
- added C24: 0.047uF, Capacitor_SMD:C_0603_1608Metric, F.Cu at (203.8, 159.3)
- added C25: 22uF, Capacitor_SMD:C_0805_2012Metric, F.Cu at (195.2, 161.7)
- added C26: 22uF, PCM_fab:C_0603, F.Cu at (186.7, 162.0)
- added C27: 22uF, Capacitor_SMD:C_0805_2012Metric, F.Cu at (199.6, 149.6)
- added C28: 22uF, Capacitor_SMD:C_0805_2012Metric, F.Cu at (199.6, 152.7)
- added C29: 47uF, Capacitor_SMD:C_0805_2012Metric, F.Cu at (195.2, 152.7)
- added C30: 0.1uF, PCM_fab:C_0603, F.Cu at (186.7, 157.0)
- added C31: 0.1uF, Capacitor_SMD:C_0805_2012Metric, F.Cu at (190.7, 152.7)
- added C32: 22uF, PCM_fab:C_0603, F.Cu at (186.7, 149.4)
- added C33: 22uF, PCM_fab:C_0603, F.Cu at (186.7, 151.9)
- added C34: 56pF, Capacitor_SMD:C_0805_2012Metric, F.Cu at (190.7, 149.6)
- added C35: 22uF, PCM_fab:C_0603, F.Cu at (186.7, 154.4)
- added C36: 47uF, Capacitor_SMD:C_0805_2012Metric, F.Cu at (190.7, 155.7)
- added C37: 47uF, Capacitor_SMD:C_0805_2012Metric, F.Cu at (190.7, 158.7)
- added C38: 47uF, Capacitor_SMD:C_0805_2012Metric, F.Cu at (190.7, 161.7)
- added C39: 47uF, Capacitor_SMD:C_0805_2012Metric, F.Cu at (195.2, 149.6)
- added L1: IHLP2525CZER2R2M01, easyeda_imports:IND-SMD_L6.5-W6.5_IHLP-2525, F.Cu at (193.1, 167.1)
- added R10: 52.3k, PCM_Resistor_SMD_AKL:R_0603_1608Metric, F.Cu at (182.8, 163.1)
- added R11: 10k, PCM_Resistor_SMD_AKL:R_0603_1608Metric, F.Cu at (182.8, 157.7)
- added R12: 10k, PCM_Resistor_SMD_AKL:R_0603_1608Metric, F.Cu at (182.8, 160.4)
- added R13: 54.9k, PCM_Resistor_SMD_AKL:R_0603_1608Metric, F.Cu at (182.8, 152.2)
- added R14: 10k, PCM_Resistor_SMD_AKL:R_0603_1608Metric, F.Cu at (182.8, 154.9)
- added R8: 49.9k, PCM_Resistor_SMD_AKL:R_0603_1608Metric, F.Cu at (182.8, 165.8)
- added R9: 10k, PCM_Resistor_SMD_AKL:R_0603_1608Metric, F.Cu at (182.8, 149.5)
- added U10: WS2812B, easyeda_imports:LED-SMD_4P-L4.0-W1.7-R, F.Cu at (183.3, 94.6)
- added U11: WS2812B, easyeda_imports:LED-SMD_4P-L4.0-W1.7-R, F.Cu at (183.3, 106.8)
- added U12: WS2812B, easyeda_imports:LED-SMD_4P-L4.0-W1.7-R, F.Cu at (188.4, 91.6)
- added U13: WS2812B, easyeda_imports:LED-SMD_4P-L4.0-W1.7-R, F.Cu at (188.4, 103.8)
- added U14: WS2812B, easyeda_imports:LED-SMD_4P-L4.0-W1.7-R, F.Cu at (188.4, 113.0)
- added U15: WS2812B, easyeda_imports:LED-SMD_4P-L4.0-W1.7-R, F.Cu at (183.3, 97.7)
- added U16: WS2812B, easyeda_imports:LED-SMD_4P-L4.0-W1.7-R, F.Cu at (183.3, 109.9)
- added U17: WS2812B, easyeda_imports:LED-SMD_4P-L4.0-W1.7-R, F.Cu at (188.4, 94.6)
- added U18: WS2812B, easyeda_imports:LED-SMD_4P-L4.0-W1.7-R, F.Cu at (188.4, 106.8)
- added U19: WS2812B, easyeda_imports:LED-SMD_4P-L4.0-W1.7-R, F.Cu at (198.7, 116.0)
- added U20: WS2812B, easyeda_imports:LED-SMD_4P-L4.0-W1.7-R, F.Cu at (183.3, 100.7)
- added U21: WS2812B, easyeda_imports:LED-SMD_4P-L4.0-W1.7-R, F.Cu at (183.3, 113.0)
- added U22: WS2812B, easyeda_imports:LED-SMD_4P-L4.0-W1.7-R, F.Cu at (188.4, 97.7)
- added U23: WS2812B, easyeda_imports:LED-SMD_4P-L4.0-W1.7-R, F.Cu at (188.4, 109.9)
- added U24: WS2812B, easyeda_imports:LED-SMD_4P-L4.0-W1.7-R, F.Cu at (203.9, 91.6)
- added U25: WS2812B, easyeda_imports:LED-SMD_4P-L4.0-W1.7-R, F.Cu at (203.9, 94.6)
- added U26: WS2812B, easyeda_imports:LED-SMD_4P-L4.0-W1.7-R, F.Cu at (203.9, 97.7)
- added U27: WS2812B, easyeda_imports:LED-SMD_4P-L4.0-W1.7-R, F.Cu at (203.9, 100.7)
- added U28: WS2812B, easyeda_imports:LED-SMD_4P-L4.0-W1.7-R, F.Cu at (203.9, 103.8)
- added U29: WS2812B, easyeda_imports:LED-SMD_4P-L4.0-W1.7-R, F.Cu at (193.6, 97.7)
- added U30: WS2812B, easyeda_imports:LED-SMD_4P-L4.0-W1.7-R, F.Cu at (188.4, 116.0)
- added U31: WS2812B, easyeda_imports:LED-SMD_4P-L4.0-W1.7-R, F.Cu at (193.6, 106.8)
- added U32: WS2812B, easyeda_imports:LED-SMD_4P-L4.0-W1.7-R, F.Cu at (203.9, 106.8)
- added U33: WS2812B, easyeda_imports:LED-SMD_4P-L4.0-W1.7-R, F.Cu at (193.6, 100.7)
- added U34: WS2812B, easyeda_imports:LED-SMD_4P-L4.0-W1.7-R, F.Cu at (193.6, 91.6)
- added U35: WS2812B, easyeda_imports:LED-SMD_4P-L4.0-W1.7-R, F.Cu at (193.6, 109.9)
- added U36: WS2812B, easyeda_imports:LED-SMD_4P-L4.0-W1.7-R, F.Cu at (193.6, 103.8)
- added U37: WS2812B, easyeda_imports:LED-SMD_4P-L4.0-W1.7-R, F.Cu at (193.6, 94.6)
- added U38: WS2812B, easyeda_imports:LED-SMD_4P-L4.0-W1.7-R, F.Cu at (193.6, 113.0)
- added U39: WS2812B, easyeda_imports:LED-SMD_4P-L4.0-W1.7-R, F.Cu at (193.6, 116.0)
- added U40: WS2812B, easyeda_imports:LED-SMD_4P-L4.0-W1.7-R, F.Cu at (198.7, 97.7)
- added U41: WS2812B, easyeda_imports:LED-SMD_4P-L4.0-W1.7-R, F.Cu at (198.7, 106.8)
- added U42: WS2812B, easyeda_imports:LED-SMD_4P-L4.0-W1.7-R, F.Cu at (198.7, 91.6)
- added U43: WS2812B, easyeda_imports:LED-SMD_4P-L4.0-W1.7-R, F.Cu at (198.7, 100.7)
- added U44: WS2812B, easyeda_imports:LED-SMD_4P-L4.0-W1.7-R, F.Cu at (198.7, 109.9)
- added U45: WS2812B, easyeda_imports:LED-SMD_4P-L4.0-W1.7-R, F.Cu at (198.7, 94.6)
- added U46: WS2812B, easyeda_imports:LED-SMD_4P-L4.0-W1.7-R, F.Cu at (198.7, 103.8)
- added U47: WS2812B, easyeda_imports:LED-SMD_4P-L4.0-W1.7-R, F.Cu at (198.7, 113.0)
- added U48: TPS562200DDCR, easyeda_imports:SOT-23-6_L2.9-W1.6-P0.95-LS2.8-BR, F.Cu at (204.2, 155.7)
- added U49: TPS568215RNNR, easyeda_imports:VQFN-HR-18_L3.5-W3.5-P0.55-BL_TPS56C215RNNR, F.Cu at (170.9, 156.2)
- added U50: CYA0630-4.7UH, easyeda_imports:IND-SMD_L7.2-W6.6_GPSR07X0, F.Cu at (202.3, 167.1)
- added U6: WS2812B, easyeda_imports:LED-SMD_4P-L4.0-W1.7-R, F.Cu at (183.3, 91.6)
- added U7: WS2812B, easyeda_imports:LED-SMD_4P-L4.0-W1.7-R, F.Cu at (183.3, 103.8)
- added U8: WS2812B, easyeda_imports:LED-SMD_4P-L4.0-W1.7-R, F.Cu at (183.3, 116.0)
- added U9: WS2812B, easyeda_imports:LED-SMD_4P-L4.0-W1.7-R, F.Cu at (188.4, 100.7)
- C11, C9: value 100nF -> 1uF
- C14, C15: value 1uF -> 100nF
- C16, C17: value 2.2uF -> 100nF
- C5: value 100nF -> RVT1C102M1010; footprint PCM_fab:C_0603 -> easyeda_imports:CAP-SMD_BD10.0-L10.3-W10.3-LS11.3-FD
- C6, C7: value 100nF -> 2.2uF
- SW12, SW13, SW14, SW15, SW9: value CPG151101D212 -> EC11E15244G1; footprint easyeda_imports:KEY-TH_CPG151101D21X -> easyeda_imports:SW-TH_EC11E15244G1
- SW2, SW3, SW5, SW6, SW7: value EC11E15244G1 -> CPG151101D212; footprint easyeda_imports:SW-TH_EC11E15244G1 -> easyeda_imports:KEY-TH_CPG151101D21X
- U4: value HC-FPC-0.5-40P-FH20 -> PT4103B23F; footprint easyeda_imports:FPC-SMD_40P-P0.50_HC-FPC-0.5-40P-FH20 -> easyeda_imports:SOT-23-6_L2.9-W1.6-P0.95-LS2.8-BR
- U5: value PT4103B23F -> HC-FPC-0.5-40P-FH20; footprint easyeda_imports:SOT-23-6_L2.9-W1.6-P0.95-LS2.8-BR -> easyeda_imports:FPC-SMD_40P-P0.50_HC-FPC-0.5-40P-FH20
- moved SW15 547.5 mm to (171.6, 76.8)
- moved SW9 546.9 mm to (114.4, 76.8)
- moved SW13 546.5 mm to (143.0, 76.8)
- moved SW14 529.5 mm to (157.3, 76.8)
- moved SW12 528.8 mm to (128.7, 76.8)
- moved C8 476.4 mm to (201.1, 69.4)
- moved SW8 475.0 mm to (151.3, 137.2)
- moved SW11 472.3 mm to (151.3, 154.1)
- moved C11 471.6 mm to (208.4, 69.4)
- moved C6 469.4 mm to (208.4, 71.9)
- moved C7 469.4 mm to (208.4, 74.4)
- moved C9 469.1 mm to (204.7, 79.5)
- moved SW1 468.8 mm to (202.4, 82.9)
- moved U3 468.8 mm to (190.0, 77.4)
- moved R4 468.8 mm to (131.1, 91.3)
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Connections:
- net /mcu/D+ renamed /mcu/USB_D+
- net /mcu/D- renamed /mcu/USB_D-
- net /mcu/D0 renamed /mcu/FSMC_D0
- net /mcu/D1 renamed /mcu/FSMC_D1
- net /mcu/D10 renamed /mcu/FSMC_D10
- net /mcu/D11 renamed /mcu/FSMC_D11
- net /mcu/D12 renamed /mcu/FSMC_D12
- net /mcu/D13 renamed /mcu/FSMC_D13
- net /mcu/D14 renamed /mcu/FSMC_D14
- net /mcu/D15 renamed /mcu/FSMC_D15
- net /mcu/D2 renamed /mcu/FSMC_D2
- net /mcu/D3 renamed /mcu/FSMC_D3
- net /mcu/D4 renamed /mcu/FSMC_D4
- net /mcu/D5 renamed /mcu/FSMC_D5
- net /mcu/D6 renamed /mcu/FSMC_D6
- net /mcu/D7 renamed /mcu/FSMC_D7
- net /mcu/D8 renamed /mcu/FSMC_D8
- net /mcu/D9 renamed /mcu/FSMC_D9
- net /mcu/LCS_CS renamed /mcu/FSMC_NE1
- net /mcu/LCS_RD renamed /mcu/FSMC_NOE
- net /mcu/LCS_RS renamed /mcu/FSMC_A16
- net /mcu/LCS_RST renamed /mcu/LCD_RST
- net /mcu/LCS_WR renamed /mcu/FSMC_NWE
- net /power-usb/D+ renamed /power-usb/USB_D+
- net /power-usb/D- renamed /power-usb/USB_D-
- C1 pad 1: /power-usb/5V_SYS -> /power-usb/+5V_SYS
- C10 pad 1: /mcu/3.3V_MCU -> /mcu/+3.3V_DIGITAL
- C11 pad 1: /mcu/3.3V_MCU -> /mcu/+3.3V_DIGITAL
- C12 pad 1: /mcu/3.3V_MCU -> /mcu/+3.3V_DIGITAL
- C13 pad 1: /mcu/3.3V_MCU -> /mcu/+3.3V_DIGITAL
- C14 pad 1: /mcu/3.3V_MCU -> /mcu/+3.3V_DIGITAL
- C15 pad 1: /mcu/3.3V_MCU -> /mcu/+3.3V_DIGITAL
- C16 pad 1: GND -> /mcu/+3.3V_DIGITAL
- C16 pad 2: Net-(U3-VCAP_1) -> GND
- C17 pad 1: GND -> /mcu/+3.3V_DIGITAL
- C17 pad 2: Net-(U3-VCAP_2) -> GND
- C2 pad 1: /power-usb/3.3V_MCU -> /power-usb/+5V_SYS
- C3 pad 1: /power-usb/5V_SYS -> /power-usb/+3.3V_DIGITAL
- C4 pad 1: /power-usb/3.3V_SYS -> /power-usb/+3.3V_DIGITAL
- C5 pad 1: /mcu/3.3V_MCU -> /power-usb/+12V
- C6 pad 1: /mcu/3.3V_MCU -> GND
- C6 pad 2: GND -> Net-(U3-VCAP_1)
- C7 pad 1: /mcu/3.3V_MCU -> GND
- C7 pad 2: GND -> Net-(U3-VCAP_2)
- C8 pad 1: /mcu/3.3V_MCU -> /mcu/+3.3V_DIGITAL
- C9 pad 1: /mcu/3.3V_MCU -> /mcu/+3.3V_DIGITAL
- D1 pad 2: /power-usb/5V_BUCK -> /power-usb/+5V_SYS
- D1 pad 3: /power-usb/5V_SYS -> /power-usb/+5V_SYS
- J2 pad 1: /power-usb/12V -> /power-usb/+12V
- R4 pad 2: unconnected-(R4-Pad2) -> /button-encoder/FADER_1
- R5 pad 2: unconnected-(R5-Pad2) -> /button-encoder/FADER_2
- R5 pad 4: unconnected-(R5-Pad4) -> (no net)
- R5 pad 5: unconnected-(R5-Pad5) -> (no net)
- R5 pad 6: unconnected-(R5-Pad6) -> (no net)
- R5 pad 7: unconnected-(R5-Pad7) -> (no net)
- R6 pad 2: unconnected-(R6-Pad2) -> /button-encoder/FADER_3
- R6 pad 4: unconnected-(R6-Pad4) -> (no net)
- R6 pad 5: unconnected-(R6-Pad5) -> (no net)
- R6 pad 6: unconnected-(R6-Pad6) -> (no net)
- R6 pad 7: unconnected-(R6-Pad7) -> (no net)
- R7 pad 2: unconnected-(R7-Pad2) -> /button-encoder/FADER_4
- R7 pad 4: unconnected-(R7-Pad4) -> (no net)
- R7 pad 5: unconnected-(R7-Pad5) -> (no net)
- R7 pad 6: unconnected-(R7-Pad6) -> (no net)
- R7 pad 7: unconnected-(R7-Pad7) -> (no net)
- SW1 pad 3: /mcu/3.3V_MCU -> /mcu/+3.3V_DIGITAL
- SW1 pad 4: /mcu/3.3V_MCU -> /mcu/+3.3V_DIGITAL
- SW10 pad 1: unconnected-(SW10-Pad1) -> /button-encoder/SW_7
- SW10 pad 2: unconnected-(SW10-Pad2) -> GND
- SW11 pad 1: unconnected-(SW11-Pad1) -> /button-encoder/SW_8
- SW11 pad 2: unconnected-(SW11-Pad2) -> GND
- SW4 pad A: unconnected-(SW4-PadA) -> /button-encoder/ENC1_A
- SW4 pad B: unconnected-(SW4-PadB) -> /button-encoder/ENC1_B
- SW4 pad D: unconnected-(SW4-PadD) -> GND
- SW4 pad E: unconnected-(SW4-PadE) -> /button-encoder/ENC1_SW
- SW8 pad 1: unconnected-(SW8-Pad1) -> /button-encoder/SW_6
- SW8 pad 2: unconnected-(SW8-Pad2) -> GND
- U1 pad 1: /power-usb/5V_SYS -> /power-usb/+5V_SYS
- U1 pad 3: /power-usb/5V_SYS -> /power-usb/+5V_SYS
- U1 pad 5: /power-usb/3.3V_MCU -> /power-usb/+3.3V_DIGITAL
- U2 pad 1: /power-usb/5V_SYS -> /power-usb/+5V_SYS
- U2 pad 3: /power-usb/5V_SYS -> /power-usb/+5V_SYS
- U2 pad 5: /power-usb/3.3V_SYS -> /power-usb/+3.3V_DIGITAL
- U3 pad 1: unconnected-(U3-PE2-Pad1) -> /mcu/ENC4_SW
- U3 pad 100: /mcu/3.3V_MCU -> /mcu/+3.3V_DIGITAL
- U3 pad 11: /mcu/3.3V_MCU -> /mcu/+3.3V_DIGITAL
- U3 pad 15: unconnected-(U3-PC0-Pad15) -> /mcu/SW_1
- U3 pad 16: unconnected-(U3-PC1-Pad16) -> /mcu/SW_2
- U3 pad 17: unconnected-(U3-PC2-Pad17) -> /mcu/SW_3
- U3 pad 18: unconnected-(U3-PC3-Pad18) -> /mcu/SW_4
- U3 pad 19: /mcu/3.3V_MCU -> /mcu/+3.3V_DIGITAL
- U3 pad 2: unconnected-(U3-PE3-Pad2) -> /mcu/ENC5_A
- U3 pad 22: /mcu/3.3V_MCU -> /mcu/+3.3V_DIGITAL
- U3 pad 28: /mcu/3.3V_MCU -> /mcu/+3.3V_DIGITAL
- U3 pad 29: unconnected-(U3-PA4-Pad29) -> /mcu/LED_ENC6_DATA
- U3 pad 3: unconnected-(U3-PE4-Pad3) -> /mcu/ENC5_B
- U3 pad 33: unconnected-(U3-PC4-Pad33) -> /mcu/SW_5
- U3 pad 35: unconnected-(U3-PB0-Pad35) -> /mcu/ENC1_A
- U3 pad 36: unconnected-(U3-PB1-Pad36) -> /mcu/ENC1_B
- U3 pad 37: unconnected-(U3-PB2-Pad37) -> /mcu/ENC1_SW
- U3 pad 4: unconnected-(U3-PE5-Pad4) -> /mcu/ENC5_SW
- U3 pad 47: unconnected-(U3-PB10-Pad47) -> /mcu/LED_FADER1_DATA
- U3 pad 48: unconnected-(U3-PB11-Pad48) -> /mcu/LED_FADER2_DATA
- U3 pad 50: /mcu/3.3V_MCU -> /mcu/+3.3V_DIGITAL
- U3 pad 51: unconnected-(U3-PB12-Pad51) -> /mcu/LED_FADER3_DATA
- U3 pad 52: unconnected-(U3-PB13-Pad52) -> /mcu/LED_FADER4_DATA
- U3 pad 59: unconnected-(U3-PD12-Pad59) -> /mcu/LED_ENC4_DATA
- U3 pad 6: /mcu/3.3V_MCU -> /mcu/+3.3V_DIGITAL
- U3 pad 60: unconnected-(U3-PD13-Pad60) -> /mcu/LED_ENC5_DATA
- U3 pad 63: unconnected-(U3-PC6-Pad63) -> /mcu/SW_6
- U3 pad 64: unconnected-(U3-PC7-Pad64) -> /mcu/SW_7
- U3 pad 65: unconnected-(U3-PC8-Pad65) -> /mcu/ENC6_A
- U3 pad 66: unconnected-(U3-PC9-Pad66) -> /mcu/ENC6_B
- U3 pad 67: unconnected-(U3-PA8-Pad67) -> /mcu/LED_KEYS_DATA
- U3 pad 75: /mcu/3.3V_MCU -> /mcu/+3.3V_DIGITAL
- U3 pad 78: unconnected-(U3-PC10-Pad78) -> /mcu/ENC6_SW
- U3 pad 79: unconnected-(U3-PC11-Pad79) -> /mcu/SW_8
- U3 pad 83: unconnected-(U3-PD2-Pad83) -> /mcu/LED_ENC1_DATA
- U3 pad 84: unconnected-(U3-PD3-Pad84) -> /mcu/LED_ENC2_DATA
- U3 pad 87: unconnected-(U3-PD6-Pad87) -> /mcu/LED_ENC3_DATA
- U3 pad 90: unconnected-(U3-PB4-Pad90) -> /mcu/ENC2_A
- U3 pad 91: unconnected-(U3-PB5-Pad91) -> /mcu/ENC2_B
- U3 pad 92: unconnected-(U3-PB6-Pad92) -> /mcu/ENC2_SW
- U3 pad 93: unconnected-(U3-PB7-Pad93) -> /mcu/ENC3_A
- U3 pad 95: unconnected-(U3-PB8-Pad95) -> /mcu/ENC3_B
- U3 pad 96: unconnected-(U3-PB9-Pad96) -> /mcu/ENC3_SW
- U3 pad 97: unconnected-(U3-PE0-Pad97) -> /mcu/ENC4_A
- U3 pad 98: unconnected-(U3-PE1-Pad98) -> /mcu/ENC4_B
- U4 pad 2: unconnected-(U4-Pad2) -> GND
- U4 pad 4: unconnected-(U4-Pad4) -> /display/+3.3V_DIGITAL
- U4 pad 6: GND -> /display/+5V_SYS
- U5 pad 2: GND -> unconnected-(U5-Pad2)
- U5 pad 4: /display/3.3V_SYS -> unconnected-(U5-Pad4)
- U5 pad 5: unconnected-(U5-OV-Pad5) -> GND
- U5 pad 6: /display/5V_SYS -> GND

Commit message: sdadsa
Parts:
- removed D2: PMEG4005CT, PCM_Package_TO_SOT_SMD_AKL:SOT-23
- removed U5: HC-FPC-0.5-40P-FH20, easyeda_imports:FPC-SMD_40P-P0.50_HC-FPC-0.5-40P-FH20
- added C40: 1uF, PCM_fab:C_0603, F.Cu at (75.3, 157.7)
- added C41: 1uF, PCM_fab:C_0603, F.Cu at (75.3, 160.2)
- added R15: 10k, Resistor_SMD:R_0603_1608Metric, F.Cu at (136.0, 148.5)
- added SW16: SKRPACE010, easyeda_imports:KEY-SMD_4P-L4.2-W3.2-P2.20-LS4.6, F.Cu at (137.1, 145.1)
- added U51: MIC5219-3.3YM5, Package_TO_SOT_SMD:SOT-23-5, F.Cu at (79.7, 158.0)
- U4: value PT4103B23F -> HS35B01A; footprint easyeda_imports:SOT-23-6_L2.9-W1.6-P0.95-LS2.8-BR -> easyeda_imports:LCD-TH_L96.5-W57.3_HS35B01A
- moved C5 127.1 mm to (80.7, 167.3)
- moved J2 122.9 mm to (66.5, 148.7)
- moved J1 122.9 mm to (66.8, 168.7)
- moved C4 121.6 mm to (75.3, 155.2)
- moved U2 121.5 mm to (79.7, 153.4)
- moved C2 121.2 mm to (75.3, 150.2)
- moved R1 120.8 mm to (84.3, 147.6)
- moved R2 120.8 mm to (84.3, 150.1)
- moved C3 120.5 mm to (75.3, 152.7)
- moved U1 120.3 mm to (79.7, 148.8)
- moved C1 120.3 mm to (75.3, 147.6)
- moved U4 117.6 mm to (178.0, 94.5)
- moved D1 115.2 mm to (84.6, 153.8)
- moved U3 102.3 mm to (142.4, 167.9)
- moved C27 100.2 mm to (100.0, 159.9)
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Connections:
- R4 pad 1: unconnected-(R4-Pad1) -> /button-encoder/+3.3V_ANALOG
- R4 pad 3: unconnected-(R4-Pad3) -> GND
- R5 pad 1: unconnected-(R5-Pad1) -> /button-encoder/+3.3V_ANALOG
- R5 pad 3: unconnected-(R5-Pad3) -> GND
- R6 pad 1: unconnected-(R6-Pad1) -> /button-encoder/+3.3V_ANALOG
- R6 pad 3: unconnected-(R6-Pad3) -> GND
- R7 pad 1: unconnected-(R7-Pad1) -> /button-encoder/+3.3V_ANALOG
- R7 pad 3: unconnected-(R7-Pad3) -> GND
- U3 pad 14: unconnected-(U3-NRST-Pad14) -> Net-(U3-NRST)
- U3 pad 21: unconnected-(U3-VREF+-Pad21) -> /mcu/+3.3V_DIGITAL
- U3 pad 94: unconnected-(U3-BOOT0-Pad94) -> /mcu/BOOT0
- U4 pad 1: unconnected-(U4-SW-Pad1) -> /display/FSMC_NE1
- U4 pad 2: GND -> /display/FSMC_A16
- U4 pad 3: unconnected-(U4-FB-Pad3) -> /display/FSMC_NWE
- U4 pad 4: /display/+3.3V_DIGITAL -> /display/FSMC_NOE
- U4 pad 5: unconnected-(U4-OV-Pad5) -> /display/LCD_RST
- U4 pad 6: /display/+5V_SYS -> /display/FSMC_D0

Commit message: holy larp is that you
holy larp is that you
Connections:
- net /bec/EN renamed EN
- net /button-encoder/FADER_1 renamed FADER_1
- net /button-encoder/FADER_2 renamed FADER_2
- net /button-encoder/FADER_3 renamed FADER_3
- net /button-encoder/FADER_4 renamed FADER_4
- net /display/BACKLIGHT_PWM renamed BACKLIGHT_PWM
- net /mcu/BOOT0 renamed BOOT0
- net /mcu/FSMC_D12 renamed FSMC_D12
- net /mcu/LED_ENC6_DATA renamed LED_ENC6_DATA
- net /mcu/SWCLK renamed SWCLK
- net /mcu/SWDIO renamed SWDIO
- net /power-usb/5V_USB renamed 5V_USB
- net /power-usb/CC1 renamed CC1
- net /power-usb/CC2 renamed CC2
- C1 pad 1: /power-usb/+5V_SYS -> +5V_SYS
- C10 pad 1: /mcu/+3.3V_DIGITAL -> +3.3V_DIGITAL
- C11 pad 1: /mcu/+3.3V_DIGITAL -> +3.3V_DIGITAL
- C12 pad 1: /mcu/+3.3V_DIGITAL -> +3.3V_DIGITAL
- C13 pad 1: /mcu/+3.3V_DIGITAL -> +3.3V_DIGITAL
- C14 pad 1: /mcu/+3.3V_DIGITAL -> +3.3V_DIGITAL
- C15 pad 1: /mcu/+3.3V_DIGITAL -> +3.3V_DIGITAL
- C16 pad 1: /mcu/+3.3V_DIGITAL -> +3.3V_DIGITAL
- C17 pad 1: /mcu/+3.3V_DIGITAL -> +3.3V_DIGITAL
- C18 pad 1: /mcu/+3.3V_DIGITAL -> +3.3V_DIGITAL
- C19 pad 2: /bec/+12V -> +12V
- C2 pad 1: /power-usb/+5V_SYS -> +5V_SYS
- C20 pad 1: /bec/+12V -> +12V
- C21 pad 2: /bec/+12V -> +12V
- C22 pad 1: /bec/+12V -> +12V
- C23 pad 2: /bec/+12V -> +12V
- C25 pad 2: /bec/+12V -> +12V
- C26 pad 1: /bec/+12V -> +12V
- C27 pad 2: /bec/+12V -> +12V
- C28 pad 2: /bec/+12V -> +12V
- C3 pad 1: /power-usb/+3.3V_DIGITAL -> +3.3V_DIGITAL
- C32 pad 1: /bec/+5V_SYS -> +5V_SYS
- C33 pad 1: /bec/+5V_SYS -> +5V_SYS
- C35 pad 1: /bec/+5V_SYS -> +5V_SYS
- C36 pad 2: /bec/+5V_LED -> +5V_LED
- C37 pad 2: /bec/+5V_LED -> +5V_LED
- C38 pad 2: /bec/+5V_LED -> +5V_LED
- C39 pad 2: /bec/+5V_LED -> +5V_LED
- C4 pad 1: /power-usb/+3.3V_DIGITAL -> +3.3V_DIGITAL
- C40 pad 1: /power-usb/+5V_SYS -> +5V_SYS
- C41 pad 1: /power-usb/+3.3V_ANALOG -> +3.3V_ANALOG
- C5 pad 1: /power-usb/+12V -> +12V
- C8 pad 1: /mcu/+3.3V_DIGITAL -> +3.3V_DIGITAL
- C9 pad 1: /mcu/+3.3V_DIGITAL -> +3.3V_DIGITAL
- D1 pad 2: /power-usb/+5V_SYS -> +5V_SYS
- D1 pad 3: /power-usb/+5V_SYS -> +5V_SYS
- J1 pad A6: /power-usb/USB_D+ -> USB_D+
- J1 pad A7: /power-usb/USB_D- -> USB_D-
- J1 pad B6: /power-usb/USB_D+ -> USB_D+
- J1 pad B7: /power-usb/USB_D- -> USB_D-
- J2 pad 1: /power-usb/+12V -> +12V
- L1 pad 2: /bec/+5V_LED -> +5V_LED
- R13 pad 2: /bec/+5V_SYS -> +5V_SYS
- R15 pad 2: /mcu/+3.3V_DIGITAL -> +3.3V_DIGITAL
- R4 pad 1: /button-encoder/+3.3V_ANALOG -> +3.3V_ANALOG
- R5 pad 1: /button-encoder/+3.3V_ANALOG -> +3.3V_ANALOG
- R6 pad 1: /button-encoder/+3.3V_ANALOG -> +3.3V_ANALOG
- R7 pad 1: /button-encoder/+3.3V_ANALOG -> +3.3V_ANALOG
- SW1 pad 3: /mcu/+3.3V_DIGITAL -> +3.3V_DIGITAL
- SW1 pad 4: /mcu/+3.3V_DIGITAL -> +3.3V_DIGITAL
- SW10 pad 1: /button-encoder/SW_7 -> SW_7
- SW11 pad 1: /button-encoder/SW_8 -> SW_8
- SW12 pad A: /button-encoder/ENC3_A -> ENC3_A
- SW12 pad B: /button-encoder/ENC3_B -> ENC3_B
- SW12 pad E: /button-encoder/ENC3_SW -> ENC3_SW
- SW13 pad A: /button-encoder/ENC4_A -> ENC4_A
- SW13 pad B: /button-encoder/ENC4_B -> ENC4_B
- SW13 pad E: /button-encoder/ENC4_SW -> ENC4_SW
- SW14 pad A: /button-encoder/ENC5_A -> ENC5_A
- SW14 pad B: /button-encoder/ENC5_B -> ENC5_B
- SW14 pad E: /button-encoder/ENC5_SW -> ENC5_SW
- SW15 pad A: /button-encoder/ENC6_A -> ENC6_A
- SW15 pad B: /button-encoder/ENC6_B -> ENC6_B
- SW15 pad E: /button-encoder/ENC6_SW -> ENC6_SW
- SW2 pad 1: /button-encoder/SW_1 -> SW_1
- SW3 pad 1: /button-encoder/SW_2 -> SW_2
- SW4 pad A: /button-encoder/ENC1_A -> ENC1_A
- SW4 pad B: /button-encoder/ENC1_B -> ENC1_B
- SW4 pad E: /button-encoder/ENC1_SW -> ENC1_SW
- SW5 pad 1: /button-encoder/SW_3 -> SW_3
- SW6 pad 1: /button-encoder/SW_4 -> SW_4
- SW7 pad 1: /button-encoder/SW_5 -> SW_5
- SW8 pad 1: /button-encoder/SW_6 -> SW_6
- SW9 pad A: /button-encoder/ENC2_A -> ENC2_A
- SW9 pad B: /button-encoder/ENC2_B -> ENC2_B
- SW9 pad E: /button-encoder/ENC2_SW -> ENC2_SW
- U1 pad 1: /power-usb/+5V_SYS -> +5V_SYS
- U1 pad 3: /power-usb/+5V_SYS -> +5V_SYS
- U1 pad 5: /power-usb/+3.3V_DIGITAL -> +3.3V_DIGITAL
- U10 pad 2: /led/+5V_LED -> +5V_LED
- U11 pad 2: /led/+5V_LED -> +5V_LED
- U12 pad 2: /led/+5V_LED -> +5V_LED
- U13 pad 2: /led/+5V_LED -> +5V_LED
- U14 pad 1: /led/LED_KEYS_DATA -> LED_KEYS_DATA
- U15 pad 2: /led/+5V_LED -> +5V_LED
- U16 pad 2: /led/+5V_LED -> +5V_LED
- U17 pad 2: /led/+5V_LED -> +5V_LED
- U18 pad 2: /led/+5V_LED -> +5V_LED
- U2 pad 1: /power-usb/+5V_SYS -> +5V_SYS
- U2 pad 3: /power-usb/+5V_SYS -> +5V_SYS
- U2 pad 5: /power-usb/+3.3V_DIGITAL -> +3.3V_DIGITAL
- U20 pad 2: /led/+5V_LED -> +5V_LED
- U21 pad 2: /led/+5V_LED -> +5V_LED
- U22 pad 2: /led/+5V_LED -> +5V_LED
- U23 pad 2: /led/+5V_LED -> +5V_LED
- U29 pad 1: /led/LED_ENC2_DATA -> LED_ENC2_DATA
- U29 pad 2: /led/+5V_LED -> +5V_LED
- U3 pad 1: /mcu/ENC4_SW -> ENC4_SW
- U3 pad 100: /mcu/+3.3V_DIGITAL -> +3.3V_DIGITAL
- U3 pad 11: /mcu/+3.3V_DIGITAL -> +3.3V_DIGITAL
- U3 pad 15: /mcu/SW_1 -> SW_1
- U3 pad 16: /mcu/SW_2 -> SW_2
- U3 pad 17: /mcu/SW_3 -> SW_3
- U3 pad 18: /mcu/SW_4 -> SW_4
- U3 pad 19: /mcu/+3.3V_DIGITAL -> +3.3V_DIGITAL
- U3 pad 2: /mcu/ENC5_A -> ENC5_A
- U3 pad 21: /mcu/+3.3V_DIGITAL -> +3.3V_DIGITAL
- U3 pad 22: /mcu/+3.3V_DIGITAL -> +3.3V_DIGITAL
- U3 pad 28: /mcu/+3.3V_DIGITAL -> +3.3V_DIGITAL
- U3 pad 3: /mcu/ENC5_B -> ENC5_B
- U3 pad 33: /mcu/SW_5 -> SW_5
- U3 pad 34: /mcu/LCD_RST -> LCD_RST
- U3 pad 35: /mcu/ENC1_A -> ENC1_A
- U3 pad 36: /mcu/ENC1_B -> ENC1_B
- U3 pad 37: /mcu/ENC1_SW -> ENC1_SW
- U3 pad 38: /mcu/FSMC_D4 -> FSMC_D4
- U3 pad 39: /mcu/FSMC_D5 -> FSMC_D5
- U3 pad 4: /mcu/ENC5_SW -> ENC5_SW
- U3 pad 40: /mcu/FSMC_D6 -> FSMC_D6
- U3 pad 41: /mcu/FSMC_D7 -> FSMC_D7
- U3 pad 42: /mcu/FSMC_D8 -> FSMC_D8
- U3 pad 43: /mcu/FSMC_D9 -> FSMC_D9
- U3 pad 44: /mcu/FSMC_D10 -> FSMC_D10
- U3 pad 45: /mcu/FSMC_D11 -> FSMC_D11
- U3 pad 47: /mcu/LED_FADER1_DATA -> LED_FADER1_DATA
- U3 pad 48: /mcu/LED_FADER2_DATA -> LED_FADER2_DATA
- U3 pad 50: /mcu/+3.3V_DIGITAL -> +3.3V_DIGITAL
- U3 pad 51: /mcu/LED_FADER3_DATA -> LED_FADER3_DATA
- U3 pad 52: /mcu/LED_FADER4_DATA -> LED_FADER4_DATA
- U3 pad 55: /mcu/FSMC_D13 -> FSMC_D13
- U3 pad 56: /mcu/FSMC_D14 -> FSMC_D14
- U3 pad 57: /mcu/FSMC_D15 -> FSMC_D15
- U3 pad 58: /mcu/FSMC_A16 -> FSMC_A16
- U3 pad 59: /mcu/LED_ENC4_DATA -> LED_ENC4_DATA
- U3 pad 6: /mcu/+3.3V_DIGITAL -> +3.3V_DIGITAL
- U3 pad 60: /mcu/LED_ENC5_DATA -> LED_ENC5_DATA
- U3 pad 61: /mcu/FSMC_D0 -> FSMC_D0
- U3 pad 62: /mcu/FSMC_D1 -> FSMC_D1
- U3 pad 63: /mcu/SW_6 -> SW_6
- U3 pad 64: /mcu/SW_7 -> SW_7
- U3 pad 65: /mcu/ENC6_A -> ENC6_A
- U3 pad 66: /mcu/ENC6_B -> ENC6_B
- U3 pad 67: /mcu/LED_KEYS_DATA -> LED_KEYS_DATA
- U3 pad 70: /mcu/USB_D- -> USB_D-
- U3 pad 71: /mcu/USB_D+ -> USB_D+
- U3 pad 75: /mcu/+3.3V_DIGITAL -> +3.3V_DIGITAL
- U3 pad 78: /mcu/ENC6_SW -> ENC6_SW
- U3 pad 79: /mcu/SW_8 -> SW_8
- U3 pad 81: /mcu/FSMC_D2 -> FSMC_D2
- U3 pad 82: /mcu/FSMC_D3 -> FSMC_D3
- U3 pad 83: /mcu/LED_ENC1_DATA -> LED_ENC1_DATA
- U3 pad 84: /mcu/LED_ENC2_DATA -> LED_ENC2_DATA
- U3 pad 85: /mcu/FSMC_NOE -> FSMC_NOE
- U3 pad 86: /mcu/FSMC_NWE -> FSMC_NWE
- U3 pad 87: /mcu/LED_ENC3_DATA -> LED_ENC3_DATA
- U3 pad 88: /mcu/FSMC_NE1 -> FSMC_NE1
- U3 pad 90: /mcu/ENC2_A -> ENC2_A
- U3 pad 91: /mcu/ENC2_B -> ENC2_B
- U3 pad 92: /mcu/ENC2_SW -> ENC2_SW
- U3 pad 93: /mcu/ENC3_A -> ENC3_A
- U3 pad 95: /mcu/ENC3_B -> ENC3_B
- U3 pad 96: /mcu/ENC3_SW -> ENC3_SW
- U3 pad 97: /mcu/ENC4_A -> ENC4_A
- U3 pad 98: /mcu/ENC4_B -> ENC4_B
- U30 pad 1: /led/LED_ENC1_DATA -> LED_ENC1_DATA
- U30 pad 2: /led/+5V_LED -> +5V_LED
- U31 pad 1: /led/LED_ENC3_DATA -> LED_ENC3_DATA
- U31 pad 2: /led/+5V_LED -> +5V_LED
- U33 pad 2: /led/+5V_LED -> +5V_LED
- U34 pad 2: /led/+5V_LED -> +5V_LED
- U35 pad 2: /led/+5V_LED -> +5V_LED
- U36 pad 2: /led/+5V_LED -> +5V_LED
- U37 pad 2: /led/+5V_LED -> +5V_LED
- U38 pad 2: /led/+5V_LED -> +5V_LED
- U39 pad 1: /led/LED_ENC3_DATA -> LED_ENC3_DATA
- U39 pad 2: /led/+5V_LED -> +5V_LED
- U4 pad 1: /display/FSMC_NE1 -> FSMC_NE1
- U4 pad 10: /display/FSMC_D4 -> FSMC_D4
- U4 pad 11: /display/FSMC_D5 -> FSMC_D5
- U4 pad 12: /display/FSMC_D6 -> FSMC_D6
- U4 pad 13: /display/FSMC_D7 -> FSMC_D7
- U4 pad 14: /display/FSMC_D8 -> FSMC_D8
- U4 pad 15: /display/FSMC_D9 -> FSMC_D9
- U4 pad 16: /display/FSMC_D10 -> FSMC_D10
- U4 pad 17: /display/FSMC_D11 -> FSMC_D11
- U4 pad 19: /display/FSMC_D13 -> FSMC_D13
- U4 pad 2: /display/FSMC_A16 -> FSMC_A16
- U4 pad 20: /display/FSMC_D14 -> FSMC_D14
- U4 pad 21: /display/FSMC_D15 -> FSMC_D15
- U4 pad 26: /display/+3.3V_DIGITAL -> +3.3V_DIGITAL
- U4 pad 3: /display/FSMC_NWE -> FSMC_NWE
- U4 pad 32: /display/+3.3V_DIGITAL -> +3.3V_DIGITAL
- U4 pad 4: /display/FSMC_NOE -> FSMC_NOE
- U4 pad 5: /display/LCD_RST -> LCD_RST
- U4 pad 6: /display/FSMC_D0 -> FSMC_D0
- U4 pad 7: /display/FSMC_D1 -> FSMC_D1
- U4 pad 8: /display/FSMC_D2 -> FSMC_D2
- U4 pad 9: /display/FSMC_D3 -> FSMC_D3
- U40 pad 1: /led/LED_ENC4_DATA -> LED_ENC4_DATA
- U40 pad 2: /led/+5V_LED -> +5V_LED
- U41 pad 1: /led/LED_ENC5_DATA -> LED_ENC5_DATA
- U41 pad 2: /led/+5V_LED -> +5V_LED
- U42 pad 2: /led/+5V_LED -> +5V_LED
- U43 pad 2: /led/+5V_LED -> +5V_LED
- U44 pad 2: /led/+5V_LED -> +5V_LED
- U45 pad 2: /led/+5V_LED -> +5V_LED
- U46 pad 2: /led/+5V_LED -> +5V_LED
- U47 pad 2: /led/+5V_LED -> +5V_LED
- U48 pad 3: /bec/+12V -> +12V
- U49 pad 11: /bec/+12V -> +12V
- U49 pad 2: /bec/+12V -> +12V
- U50 pad 2: /bec/+5V_SYS -> +5V_SYS
- U51 pad 1: /power-usb/+5V_SYS -> +5V_SYS
- U51 pad 3: /power-usb/+5V_SYS -> +5V_SYS
- U51 pad 5: /power-usb/+3.3V_ANALOG -> +3.3V_ANALOG
- U6 pad 1: /led/LED_FADER1_DATA -> LED_FADER1_DATA
- U6 pad 2: /led/+5V_LED -> +5V_LED
- U7 pad 1: /led/LED_FADER2_DATA -> LED_FADER2_DATA
- U7 pad 2: /led/+5V_LED -> +5V_LED
- U8 pad 1: /led/LED_FADER3_DATA -> LED_FADER3_DATA
- U8 pad 2: /led/+5V_LED -> +5V_LED
- U9 pad 1: /led/LED_FADER4_DATA -> LED_FADER4_DATA
- U9 pad 2: /led/+5V_LED -> +5V_LED
