File: Hardware/board/bec.kicad_sch (KiCad schematic)
At the start: 32 parts, among them U48 TPS562200DDCR, U49 TPS568215RNNR, U50 CYA0630-4.7UH

Commit message: sdadsa
Changed lines of the file:
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@@
+	)
+	(junction
+		(at 178.435 106.045)
+		(diameter 0)
+		(color 0 0 0 0)
 	)
 	(junction
@@
 	)
 	(junction
+		(at 187.325 106.045)
+		(diameter 0)
+		(color 0 0 0 0)
+	)
+	(junction
 		(at 169.545 113.665)
 		(diameter 0)
@@
 	)
 	(junction
-		(at 178.435 106.045)
-		(diameter 0)
-		(color 0 0 0 0)
-	)
-	(junction
 		(at 42.545 27.305)
 		(diameter 0)
@@
 	(wire
 		(pts
+			(xy 188.595 106.045) (xy 187.325 106.045)
+		)
+		(stroke
+			(width 0)
+			(type default)
+		)
+	)
+	(wire
+		(pts
 			(xy 60.325 104.775) (xy 68.58 104.775)
 		)
@@
 		)
 	)
-	(label "+5V_SYS"
+	(global_label "+5V_SYS"
+		(shape bidirectional)
 		(at 160.02 27.305 0)
 		(effects
@@
 				(size 1.27 1.27)
 			)
-			(justify left bottom)
-		)
-	)
-	(label "EN"
+			(justify left)
+		)
+		(property "Intersheetrefs" "${INTERSHEET_REFS}"
+			(at 160.02 27.305 0)
+			(hide yes)
+			(show_name no)
+			(do_not_autoplace no)
+			(effects
+				(font
+					(size 1.27 1.27)
+				)
+			)
+		)
+	)
+	(global_label "EN"
+		(shape bidirectional)
 		(at 65.405 29.845 180)
 		(effects
@@
 				(size 1.27 1.27)
 			)
-			(justify right bottom)
-		)
-	)
-	(label "EN"
+			(justify right)
+		)
+		(property "Intersheetrefs" "${INTERSHEET_REFS}"
+			(at 65.405 29.845 0)
+			(hide yes)
+			(show_name no)
+			(do_not_autoplace no)
+			(effects
+				(font
+					(size 1.27 1.27)
+				)
+			)
+		)
+	)
+	(global_label "EN"
+		(shape bidirectional)
 		(at 91.44 122.555 180)
 		(effects
@@
 				(size 1.27 1.27)
 			)
-			(justify right bottom)
-		)
-	)
-	(label "+5V_LED"
-		(at 187.325 106.045 0)
+			(justify right)
+		)
+		(property "Intersheetrefs" "${INTERSHEET_REFS}"
+			(at 91.44 122.555 0)
+			(hide yes)
+			(show_name no)
+			(do_not_autoplace no)
+			(effects
+				(font
+					(size 1.27 1.27)
+				)
+			)
+		)
+	)
+	(global_label "+5V_LED"
+		(shape bidirectional)
+		(at 188.595 106.045 0)
 		(effects
 			(font
 				(size 1.27 1.27)
 			)
-			(justify left bottom)
-		)
-	)
-	(label "+12V"
+			(justify left)
+		)
+		(property "Intersheetrefs" "${INTERSHEET_REFS}"
+			(at 188.595 106.045 0)
+			(hide yes)
+			(show_name no)
+			(do_not_autoplace no)
+			(effects
+				(font
+					(size 1.27 1.27)
+				)
+			)
+		)
+	)
+	(global_label "+12V"
+		(shape bidirectional)
 		(at 29.845 27.305 180)
 		(effects
@@
 				(size 1.27 1.27)
 			)
-			(justify right bottom)
-		)
-	)
-	(label "+12V"
+			(justify right)
+		)
+		(property "Intersheetrefs" "${INTERSHEET_REFS}"
+			(at 29.845 27.305 0)
+			(hide yes)
+			(show_name no)
+			(do_not_autoplace no)
+			(effects
+				(font
+					(size 1.27 1.27)
+				)
+			)
+		)
+	)
+	(global_label "+12V"
+		(shape bidirectional)
 		(at 27.305 104.775 180)
 		(effects
@@
 				(size 1.27 1.27)
 			)
-			(justify right bottom)
-		)
-	)
+			(justify right)
+		)
+		(property "Intersheetrefs" "${INTERSHEET_REFS}"
+			(at 27.305 104.775 0)
+			(hide yes)
+			(show_name no)
+			(do_not_autoplace no)
+			(effects
+				(font
+					(size 1.27 1.27)
+				)
+			)
+		)
+	)

Commit message: i am cooked
Parts:
- removed R9: 10k, PCM_Resistor_SMD_AKL:R_0603_1608Metric, symbol PCM_Resistor_US_AKL:R_0603
- added C65, C68, C72, C80, C83, C86: 22uF, Capacitor_SMD:C_1206_3216Metric, symbol PCM_fab:C_0603
- added C78: 0.1uF, PCM_SparkFun-Coil:0805, symbol PCM_fab:C_0603
- added R13: 33.2k, PCM_Resistor_SMD_AKL:R_0603_1608Metric, symbol PCM_Resistor_US_AKL:R_0603
- added R14: 10k, PCM_Resistor_SMD_AKL:R_0603_1608Metric, symbol PCM_Resistor_US_AKL:R_0603
- added U5: TPS562200DDCR, easyeda_imports:SOT-23-6_L2.9-W1.6-P0.95-LS2.8-BR, symbol easyeda_imports:TPS562200DDCR
- added U8: CYA0630-4.7UH, easyeda_imports:IND-SMD_L7.2-W6.6_GPSR07X0, symbol easyeda_imports:CYA0630-4.7UH
- C64: renamed from C19; footprint Capacitor_SMD:C_0805_2012Metric -> PCM_4ms_Capacitor:C_1206
- C66: renamed from C20; footprint PCM_fab:C_0603 -> Capacitor_SMD:C_1206_3216Metric
- C67: renamed from C21; footprint Capacitor_SMD:C_0805_2012Metric -> PCM_4ms_Capacitor:C_1206
- C69: renamed from C22; footprint PCM_fab:C_0603 -> Capacitor_SMD:C_1206_3216Metric
- C70: renamed from C23; footprint Capacitor_SMD:C_0805_2012Metric -> PCM_4ms_Capacitor:C_1206
- C73: renamed from C25; footprint Capacitor_SMD:C_0805_2012Metric -> PCM_4ms_Capacitor:C_1206
- C74: renamed from C26; footprint PCM_fab:C_0603 -> Capacitor_SMD:C_1206_3216Metric
- C75: renamed from C27; footprint Capacitor_SMD:C_0805_2012Metric -> PCM_4ms_Capacitor:C_1206
- C76: renamed from C28; footprint Capacitor_SMD:C_0805_2012Metric -> PCM_4ms_Capacitor:C_1206
- C79: renamed from C30; footprint PCM_fab:C_0603 -> PCM_SparkFun-Coil:0805
- C81: renamed from C31; footprint Capacitor_SMD:C_0805_2012Metric -> PCM_4ms_Capacitor:C_0603
- C82: renamed from C32; footprint PCM_fab:C_0603 -> Capacitor_SMD:C_1206_3216Metric
- C84: renamed from C33; footprint PCM_fab:C_0603 -> Capacitor_SMD:C_1206_3216Metric
- C87: renamed from C35; footprint PCM_fab:C_0603 -> Capacitor_SMD:C_1206_3216Metric
- C88: renamed from C36; footprint Capacitor_SMD:C_0805_2012Metric -> PCM_4ms_Capacitor:C_1206
- C89: renamed from C37; footprint Capacitor_SMD:C_0805_2012Metric -> PCM_4ms_Capacitor:C_1206
- C90: renamed from C38; footprint Capacitor_SMD:C_0805_2012Metric -> PCM_4ms_Capacitor:C_1206
- C91: renamed from C39; footprint Capacitor_SMD:C_0805_2012Metric -> PCM_4ms_Capacitor:C_1206
- L43: renamed from L1; value IHLP2525CZER2R2M01 -> WS2812B; footprint easyeda_imports:IND-SMD_L6.5-W6.5_IHLP-2525 -> easyeda_imports:LED-SMD_4P-L2.0-W2.0-TL_WS2812B-2020; LCSC Part C540967 -> C965555; MPN IHLP2525CZER2R2M01 -> WS2812B-2020; Manufacturer VISHAY(威世) -> worldsemi
- renumbered C24 to C71, C29 to C77, C34 to C85, R13 to R15, R14 to R16, R8 to R9, U48 to U6, U49 to U7, U50 to U9
Connections:
- net +12V: now also U6.5 (EN), C65.1, C68.1, C72.1, U5.3 (VIN), U5.5 (EN)
- net +5V_LED: now also C85.2, R12.1; no longer L43.2
- net GND: now also C65.2, C68.2, C72.2, C80.2, C83.2, C86.2, R14.1, U5.1 (GND)
- net at C81.2, U7.6 (SW), U7.7 (SW): no longer L43.1
- new net: R13.1, R14.2, U5.4 (VFB)
- new net: C78.1, U5.6 (VBST)
- new net: C78.2, U5.2 (SW), U8.1
- new net +3.3V_DISPLAY: C80.1, C83.1, C86.1, R13.2, U8.2

Commit message: i hate it
Parts:
- renumbered R14 to R10, R15 to R11, R16 to R12, R9 to R5, R10 to R6, R11 to R7, R12 to R8, R13 to R9
Changed lines of the file:
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@@
 		(in_pos_files yes)
 		(dnp no)
-		(property "Reference" "R13"
+		(property "Reference" "R9"
 			(at 161.29 67.31 90)
 			(show_name no)
@@
 			(project "board"
 				(path "/a701f4fd-d5c8-4ab0-b464-3edf07ec58ed/439b5fef-8eb6-4cc2-837e-59cefe4bc8c0"
-					(reference "R13")
+					(reference "R9")
 					(unit 1)
 				)
@@
 		(in_pos_files yes)
 		(dnp no)
-		(property "Reference" "R12"
+		(property "Reference" "R8"
 			(at 144.78 114.935 90)
 			(show_name no)
@@
 			(project "board"
 				(path "/a701f4fd-d5c8-4ab0-b464-3edf07ec58ed/439b5fef-8eb6-4cc2-837e-59cefe4bc8c0"
-					(reference "R12")
+					(reference "R8")
 					(unit 1)
 				)
@@
 		(in_pos_files yes)
 		(dnp no)
-		(property "Reference" "R15"
+		(property "Reference" "R11"
 			(at 162.56 34.925 90)
 			(show_name no)
@@
 			(project "board"
 				(path "/a701f4fd-d5c8-4ab0-b464-3edf07ec58ed/439b5fef-8eb6-4cc2-837e-59cefe4bc8c0"
-					(reference "R15")
+					(reference "R11")
 					(unit 1)
 				)
@@
 		(in_pos_files yes)
 		(dnp no)
-		(property "Reference" "R14"
+		(property "Reference" "R10"
 			(at 161.29 76.835 90)
 			(show_name no)
@@
 			(project "board"
 				(path "/a701f4fd-d5c8-4ab0-b464-3edf07ec58ed/439b5fef-8eb6-4cc2-837e-59cefe4bc8c0"
-					(reference "R14")
+					(reference "R10")
 					(unit 1)
 				)
@@
 		(in_pos_files yes)
 		(dnp no)
-		(property "Reference" "R10"
+		(property "Reference" "R6"
 			(at 67.945 132.715 90)
 			(show_name no)
@@
 			(project "board"
 				(path "/a701f4fd-d5c8-4ab0-b464-3edf07ec58ed/439b5fef-8eb6-4cc2-837e-59cefe4bc8c0"
-					(reference "R10")
+					(reference "R6")
 					(unit 1)
 				)
@@
 		(in_pos_files yes)
 		(dnp no)
-		(property "Reference" "R9"
+		(property "Reference" "R5"
 			(at 57.785 144.145 90)
 			(show_name no)
@@
 			(project "board"
 				(path "/a701f4fd-d5c8-4ab0-b464-3edf07ec58ed/439b5fef-8eb6-4cc2-837e-59cefe4bc8c0"
-					(reference "R9")
+					(reference "R5")
 					(unit 1)
 				)
@@
 		(in_pos_files yes)
 		(dnp no)
-		(property "Reference" "R11"
+		(property "Reference" "R7"
 			(at 135.89 132.715 90)
 			(show_name no)
@@
 			(project "board"
 				(path "/a701f4fd-d5c8-4ab0-b464-3edf07ec58ed/439b5fef-8eb6-4cc2-837e-59cefe4bc8c0"
-					(reference "R11")
+					(reference "R7")
 					(unit 1)
 				)
@@
 		(in_pos_files yes)
 		(dnp no)
-		(property "Reference" "R16"
+		(property "Reference" "R12"
 			(at 162.56 44.45 90)
 			(show_name no)
@@
 			(project "board"
 				(path "/a701f4fd-d5c8-4ab0-b464-3edf07ec58ed/439b5fef-8eb6-4cc2-837e-59cefe4bc8c0"
-					(reference "R16")
+					(reference "R12")
 					(unit 1)
 				)

Commit message: wiring and wiring
wiring and wiring
Parts:
- C64, C67, C70, C73, C75, C76, C88, C89, C90, C91: footprint PCM_4ms_Capacitor:C_1206 -> Capacitor_SMD:C_1206_3216Metric
- L43: value WS2812B -> IHLP2525CZER2R2M01; footprint easyeda_imports:LED-SMD_4P-L2.0-W2.0-TL_WS2812B-2020 -> easyeda_imports:IND-SMD_L6.5-W6.5_IHLP-2525; LCSC Part C965555 -> C540967; MPN WS2812B-2020 -> IHLP2525CZER2R2M01; Manufacturer worldsemi -> VISHAY(威世)
Connections:
- net +5V_LED: now also L43.2
- net at L43.1: now also C81.2, U7.6 (SW), U7.7 (SW)
Changed lines of the file:
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@@
 			)
 		)
-		(property "Footprint" "PCM_4ms_Capacitor:C_1206"
+		(property "Footprint" "Capacitor_SMD:C_1206_3216Metric"
 			(at 28.2702 104.775 0)
 			(hide yes)
@@
 			)
 		)
-		(property "Footprint" "PCM_4ms_Capacitor:C_1206"
+		(property "Footprint" "Capacitor_SMD:C_1206_3216Metric"
 			(at 44.7802 104.775 0)
 			(hide yes)
@@
 			)
 		)
-		(property "Footprint" "PCM_4ms_Capacitor:C_1206"
+		(property "Footprint" "Capacitor_SMD:C_1206_3216Metric"
 			(at 61.2902 104.775 0)
 			(hide yes)
@@
 			)
 		)
-		(property "Footprint" "PCM_4ms_Capacitor:C_1206"
+		(property "Footprint" "Capacitor_SMD:C_1206_3216Metric"
 			(at 36.5252 104.775 0)
 			(hide yes)
@@
 	)
 	(symbol
+		(lib_id "easyeda_imports:IHLP2525CZER2R2M01")
+		(at 146.685 106.045 0)
+		(unit 1)
+		(body_style 1)
+		(exclude_from_sim no)
+		(in_bom yes)
+		(on_board yes)
+		(in_pos_files yes)
+		(dnp no)
+		(fields_autoplaced yes)
+		(property "Reference" "L43"
+			(at 146.685 100.33 0)
+			(show_name no)
+			(do_not_autoplace no)
+			(effects
+				(font
+					(size 1.27 1.27)
+				)
+			)
+		)
+		(property "Value" "IHLP2525CZER2R2M01"
+			(at 146.685 102.87 0)
+			(show_name no)
+			(do_not_autoplace no)
+			(effects
+				(font
+					(size 1.27 1.27)
+				)
+			)
+		)
+		(property "Footprint" "easyeda_imports:IND-SMD_L6.5-W6.5_IHLP-2525"
+			(at 146.685 113.665 0)
+			(hide yes)
+			(show_name no)
+			(do_not_autoplace no)
+			(effects
+				(font
+					(size 1.27 1.27)
+				)
+			)
+		)
+		(property "Datasheet" "https://lcsc.com/product-detail/Inductors-SMD_Vishay-Intertech-IHLP2525CZER2R2M01_C540967.html"
+			(at 146.685 116.205 0)
+			(hide yes)
+			(show_name no)
+			(do_not_autoplace no)
+			(effects
+				(font
+					(size 1.27 1.27)
+				)
+			)
+		)
+		(property "Description" ""
+			(at 146.685 106.045 0)
+			(hide yes)
+			(show_name no)
+			(do_not_autoplace no)
+			(effects
+				(font
+					(size 1.27 1.27)
+				)
+			)
+		)
+		(property "Manufacturer" "VISHAY(威世)"
+			(at 146.685 118.745 0)
+			(hide yes)
+			(show_name no)
+			(do_not_autoplace no)
+			(effects
+				(font
+					(size 1.27 1.27)
+				)
+			)
+		)
+		(property "MPN" "IHLP2525CZER2R2M01"
+			(at 146.685 121.285 0)
+			(hide yes)
+			(show_name no)
+			(do_not_autoplace no)
+			(effects
+				(font
+					(size 1.27 1.27)
+				)
+			)
+		)
+		(property "LCSC Part" "C540967"
+			(at 146.685 123.825 0)
+			(hide yes)
+			(show_name no)
+			(do_not_autoplace no)
+			(effects
+				(font
+					(size 1.27 1.27)
+				)
+			)
+		)
+		(pin "2"
+		)
+		(pin "1"
+		)
+		(instances
+			(project "board"
+				(path "/a701f4fd-d5c8-4ab0-b464-3edf07ec58ed/439b5fef-8eb6-4cc2-837e-59cefe4bc8c0"
+					(reference "L43")
+					(unit 1)
+				)
+			)
+		)
+	)
+	(symbol
 		(lib_id "power:GND")
 		(at 102.235 32.385 0)
@@
 	)
 	(symbol
-		(lib_id "easyeda_imports:IHLP2525CZER2R2M01")
-		(at 146.685 106.045 0)
-		(unit 1)
-		(body_style 1)
-		(exclude_from_sim no)
-		(in_bom yes)
-		(on_board yes)
-		(in_pos_files yes)
-		(dnp no)
-		(fields_autoplaced yes)
-		(property "Reference" "L43"
-			(at 148.082 112.522 90)
-			(show_name no)
-			(do_not_autoplace no)
-			(effects
-				(font
-					(size 1.27 1.27)
-				)
-			)
-		)
-		(property "Value" "WS2812B"
-			(at 148.082 106.426 90)
-			(show_name no)
-			(do_not_autoplace no)
-			(effects
-				(font
-					(size 1.27 1.27)
-				)
-			)
-		)
-		(property "Footprint" "easyeda_imports:LED-SMD_4P-L2.0-W2.0-TL_WS2812B-2020"
-			(at 146.685 114.935 0)
-			(hide yes)
-			(show_name no)
-			(do_not_autoplace no)
-			(effects
-				(font
-					(size 1.27 1.27)
-				)
-			)
-		)
-		(property "Datasheet" "https://lcsc.com/product-detail/Light-Emitting-Diodes-LED_Worldsemi-WS2812B-2020_C965555.html"
-			(at 146.685 117.475 0)
-			(hide yes)
-			(show_name no)
-			(do_not_autoplace no)
-			(effects
-				(font
-					(size 1.27 1.27)
-				)
-			)
-		)
-		(property "Description" ""
-			(at 146.685 106.045 0)
-			(hide yes)
-			(show_name no)
-			(do_not_autoplace no)
-			(effects
-				(font
-					(size 1.27 1.27)
-				)
-			)
-		)
-		(property "Manufacturer" "worldsemi"
-			(at 146.685 120.015 0)
-			(hide yes)
-			(show_name no)
-			(do_not_autoplace no)
-			(effects
-				(font
-					(size 1.27 1.27)
-				)
-			)
-		)
-		(property "MPN" "WS2812B-2020"
-			(at 146.685 122.555 0)
-			(hide yes)
-			(show_name no)
-			(do_not_autoplace no)
-			(effects
-				(font
-					(size 1.27 1.27)
-				)
-			)
-		)
-		(property "LCSC Part" "C965555"
-			(at 146.685 125.095 0)
-			(hide yes)
-			(show_name no)
-			(do_not_autoplace no)
-			(effects
-				(font
-					(size 1.27 1.27)
-				)
-			)
-		)
-		(pin "1"
-		)
-		(pin "2"
-		)
-		(pin "4"
-		)
-		(pin "3"
-		)
-		(instances
-			(project "board"
-				(path "/a701f4fd-d5c8-4ab0-b464-3edf07ec58ed/439b5fef-8eb6-4cc2-837e-59cefe4bc8c0"
-					(reference "L43")
-					(unit 1)
-				)
-			)
-		)
-	)
-	(symbol
 		(lib_id "PCM_Capacitor_US_AKL:C_0805")
 		(at 52.07 108.585 0)
@@
 			)
 		)
-		(property "Footprint" "PCM_4ms_Capacitor:C_1206"
+		(property "Footprint" "Capacitor_SMD:C_1206_3216Metric"
 			(at 53.0352 104.775 0)
 			(hide yes)
@@
 			)
 		)
-		(property "Footprint" "PCM_4ms_Capacitor:C_1206"
+		(property "Footprint" "Capacitor_SMD:C_1206_3216Metric"
 			(at 69.5452 104.775 0)
 			(hide yes)
@@
 			)
 		)
-		(property "Footprint" "PCM_4ms_Capacitor:C_1206"
+		(property "Footprint" "Capacitor_SMD:C_1206_3216Metric"
 			(at 188.2902 106.045 0)
 			(hide yes)
@@
 			)
 		)
-		(property "Footprint" "PCM_4ms_Capacitor:C_1206"
+		(property "Footprint" "Capacitor_SMD:C_1206_3216Metric"
 			(at 179.4002 106.045 0)
 			(hide yes)
@@
 			)
 		)
-		(property "Footprint" "PCM_4ms_Capacitor:C_1206"
+		(property "Footprint" "Capacitor_SMD:C_1206_3216Metric"
 			(at 170.5102 106.045 0)
 			(hide yes)
@@
 			)
 		)
-		(property "Footprint" "PCM_4ms_Capacitor:C_1206"
+		(property "Footprint" "Capacitor_SMD:C_1206_3216Metric"
 			(at 161.6202 106.045 0)
 			(hide yes)
