File: Hardware/board/button-encoder.kicad_sch (KiCad schematic)
At the start: 18 parts, among them SW10 CPG151101D212, SW11 CPG151101D212, SW12 CPG151101D212, SW13 CPG151101D212, SW14 CPG151101D212, SW15 CPG151101D212, SW2 EC11E15244G1, SW3 EC11E15244G1, SW4 EC11E15244G1, SW5 EC11E15244G1, SW6 EC11E15244G1, SW7 EC11E15244G1, SW8 CPG151101D212, SW9 CPG151101D212

Commit message: desigin designing
dsa
Parts:
- renumbered SW11 to SW10, SW15 to SW11, SW4 to SW12, SW5 to SW13, SW6 to SW14, SW7 to SW15, SW8 to SW2, SW12 to SW3, SW2 to SW4, SW9 to SW5, SW13 to SW6, SW10 to SW7, SW14 to SW8, SW3 to SW9
Connections:
- net E1-A renamed ENC1_A
- net E1-B renamed ENC1_B
- net E1-S renamed ENC1_SW
- net E2-A renamed ENC2_A
- net E2-B renamed ENC2_B
- net E2-S renamed ENC2_SW
- net E3-A renamed ENC3_A
- net E3-B renamed ENC3_B
- net E3-S renamed ENC3_SW
- net E4-A renamed ENC4_A
- net E4-B renamed ENC4_B
- net E4-S renamed ENC4_SW
- net E5-A renamed ENC5_A
- net E5-B renamed ENC5_B
- net E5-S renamed ENC5_SW
- net E6-A renamed ENC6_A
- net E6-B renamed ENC6_B
- net E6-S renamed ENC6_SW
- net F-A1 renamed FADER_1
- net F-A2 renamed FADER_2
- net F-A3 renamed FADER_3
- net F-A4 renamed FADER_4
- net K1 renamed SW_1
- net K2 renamed SW_2
- net K3 renamed SW_3
- net K4 renamed SW_4
- net K5 renamed SW_5
- net K6 renamed SW_6
- net K7 renamed SW_7
- net K8 renamed SW_8

Commit message: sdadsa
Connections:
- net GND: now also R4.3, R5.3, R6.3, R7.3
- net +3.3V_ANALOG: now reaches R7.1
- net +3.3V_ANALOG: now also R4.1, R5.1, R6.1

Commit message: i am cooked
Parts:
- renumbered R4 to R5, R5 to R6, R6 to R7, R7 to R8, SW9 to SW10, SW10 to SW11, SW11 to SW12, SW12 to SW13, SW13 to SW14, SW14 to SW15, SW15 to SW16, SW2 to SW3, SW3 to SW4, SW4 to SW5, SW5 to SW6, SW6 to SW7, SW7 to SW8, SW8 to SW9

Commit message: i hate it
Parts:
- renumbered SW5 to EN1, SW10 to EN2, SW13 to EN3, SW14 to EN4, SW15 to EN5, SW16 to EN6, R5 to F1, R6 to F2, R7 to F3, R8 to F4, SW3 to M1, SW4 to M2, SW6 to M3, SW7 to M4, SW8 to M5, SW9 to M6, SW11 to M7, SW12 to M8
Changed lines of the file:
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@@
 		(dnp no)
 		(fields_autoplaced yes)
-		(property "Reference" "SW10"
+		(property "Reference" "EN2"
 			(at 149.86 109.7848 0)
 			(show_name no)
@@
 			(project "board"
 				(path "/a701f4fd-d5c8-4ab0-b464-3edf07ec58ed/58fefd48-2eee-4fcb-b0ad-9a73a5e36ec8"
-					(reference "SW10")
+					(reference "EN2")
 					(unit 1)
 				)
@@
 		(dnp no)
 		(fields_autoplaced yes)
-		(property "Reference" "SW14"
+		(property "Reference" "EN4"
 			(at 210.82 111.0548 0)
 			(show_name no)
@@
 			(project "board"
 				(path "/a701f4fd-d5c8-4ab0-b464-3edf07ec58ed/58fefd48-2eee-4fcb-b0ad-9a73a5e36ec8"
-					(reference "SW14")
+					(reference "EN4")
 					(unit 1)
 				)
@@
 		(dnp no)
 		(fields_autoplaced yes)
-		(property "Reference" "SW5"
-			(at 117.475 109.1498 0)
+		(property "Reference" "EN1"
+			(at 118.11 109.1498 0)
 			(show_name no)
 			(do_not_autoplace no)
@@
 		)
 		(property "Value" "EC11E15244G1"
-			(at 117.475 111.6898 0)
+			(at 118.11 111.6898 0)
 			(show_name no)
 			(do_not_autoplace no)
@@
 			(project "board"
 				(path "/a701f4fd-d5c8-4ab0-b464-3edf07ec58ed/58fefd48-2eee-4fcb-b0ad-9a73a5e36ec8"
-					(reference "SW5")
+					(reference "EN1")
 					(unit 1)
 				)
@@
 		(dnp no)
 		(fields_autoplaced yes)
-		(property "Reference" "R8"
-			(at 163.195 57.7148 0)
+		(property "Reference" "F4"
+			(at 146.56 69.85 0)
 			(show_name no)
 			(do_not_autoplace no)
@@
 		)
 		(property "Value" "PTA6043-2015CPB103"
-			(at 163.195 60.2548 0)
+			(at 146.56 72.39 0)
 			(show_name no)
 			(do_not_autoplace no)
@@
 			(project "board"
 				(path "/a701f4fd-d5c8-4ab0-b464-3edf07ec58ed/58fefd48-2eee-4fcb-b0ad-9a73a5e36ec8"
-					(reference "R8")
+					(reference "F4")
 					(unit 1)
 				)
@@
 		(dnp no)
 		(fields_autoplaced yes)
-		(property "Reference" "SW9"
+		(property "Reference" "M6"
 			(at 132.08 172.72 0)
 			(show_name no)
@@
 			(project "board"
 				(path "/a701f4fd-d5c8-4ab0-b464-3edf07ec58ed/58fefd48-2eee-4fcb-b0ad-9a73a5e36ec8"
-					(reference "SW9")
+					(reference "M6")
 					(unit 1)
 				)
@@
 		(dnp no)
 		(fields_autoplaced yes)
-		(property "Reference" "SW7"
+		(property "Reference" "M4"
 			(at 110.49 172.72 0)
 			(show_name no)
@@
 			(project "board"
 				(path "/a701f4fd-d5c8-4ab0-b464-3edf07ec58ed/58fefd48-2eee-4fcb-b0ad-9a73a5e36ec8"
-					(reference "SW7")
+					(reference "M4")
 					(unit 1)
 				)
@@
 		(dnp no)
 		(fields_autoplaced yes)
-		(property "Reference" "SW13"
-			(at 178.435 110.4198 0)
+		(property "Reference" "EN3"
+			(at 179.07 110.4198 0)
 			(show_name no)
 			(do_not_autoplace no)
@@
 		)
 		(property "Value" "EC11E15244G1"
-			(at 178.435 112.9598 0)
+			(at 179.07 112.9598 0)
 			(show_name no)
 			(do_not_autoplace no)
@@
 			(project "board"
 				(path "/a701f4fd-d5c8-4ab0-b464-3edf07ec58ed/58fefd48-2eee-4fcb-b0ad-9a73a5e36ec8"
-					(reference "SW13")
+					(reference "EN3")
 					(unit 1)
 				)
@@
 		(dnp no)
 		(fields_autoplaced yes)
-		(property "Reference" "SW3"
+		(property "Reference" "M1"
 			(at 88.9 161.29 0)
 			(show_name no)
@@
 			(project "board"
 				(path "/a701f4fd-d5c8-4ab0-b464-3edf07ec58ed/58fefd48-2eee-4fcb-b0ad-9a73a5e36ec8"
-					(reference "SW3")
+					(reference "M1")
 					(unit 1)
 				)
@@
 		(dnp no)
 		(fields_autoplaced yes)
-		(property "Reference" "SW4"
+		(property "Reference" "M2"
 			(at 88.9 172.72 0)
 			(show_name no)
@@
 			(project "board"
 				(path "/a701f4fd-d5c8-4ab0-b464-3edf07ec58ed/58fefd48-2eee-4fcb-b0ad-9a73a5e36ec8"
-					(reference "SW4")
+					(reference "M2")
 					(unit 1)
 				)
@@
 		(dnp no)
 		(fields_autoplaced yes)
-		(property "Reference" "SW12"
+		(property "Reference" "M8"
 			(at 156.845 172.72 0)
 			(show_name no)
@@
 			(project "board"
 				(path "/a701f4fd-d5c8-4ab0-b464-3edf07ec58ed/58fefd48-2eee-4fcb-b0ad-9a73a5e36ec8"
-					(reference "SW12")
+					(reference "M8")
 					(unit 1)
 				)
@@
 		(dnp no)
 		(fields_autoplaced yes)
-		(property "Reference" "SW8"
-			(at 132.08 161.925 0)
+		(property "Reference" "M5"
+			(at 132.08 161.29 0)
 			(show_name no)
 			(do_not_autoplace no)
@@
 		)
 		(property "Value" "CPG151101D212"
-			(at 132.08 164.465 0)
+			(at 132.08 163.83 0)
 			(show_name no)
 			(do_not_autoplace no)
@@
 			(project "board"
 				(path "/a701f4fd-d5c8-4ab0-b464-3edf07ec58ed/58fefd48-2eee-4fcb-b0ad-9a73a5e36ec8"
-					(reference "SW8")
+					(reference "M5")
 					(unit 1)
 				)
@@
 		(dnp no)
 		(fields_autoplaced yes)
-		(property "Reference" "R7"
-			(at 162.56 40.5698 0)
+		(property "Reference" "F3"
+			(at 145.925 53.34 0)
 			(show_name no)
 			(do_not_autoplace no)
@@
 		)
 		(property "Value" "PTA6043-2015CPB103"
-			(at 162.56 43.1098 0)
+			(at 145.925 55.88 0)
 			(show_name no)
 			(do_not_autoplace no)
@@
 			(project "board"
 				(path "/a701f4fd-d5c8-4ab0-b464-3edf07ec58ed/58fefd48-2eee-4fcb-b0ad-9a73a5e36ec8"
-					(reference "R7")
+					(reference "F3")
 					(unit 1)
 				)
@@
 		(dnp no)
 		(fields_autoplaced yes)
-		(property "Reference" "SW11"
-			(at 156.845 161.925 0)
+		(property "Reference" "M7"
+			(at 156.845 161.29 0)
 			(show_name no)
 			(do_not_autoplace no)
@@
 		)
 		(property "Value" "CPG151101D212"
-			(at 156.845 164.465 0)
+			(at 156.845 163.83 0)
 			(show_name no)
 			(do_not_autoplace no)
@@
 			(project "board"
 				(path "/a701f4fd-d5c8-4ab0-b464-3edf07ec58ed/58fefd48-2eee-4fcb-b0ad-9a73a5e36ec8"
-					(reference "SW11")
+					(reference "M7")
 					(unit 1)
 				)
@@
 		(dnp no)
 		(fields_autoplaced yes)
-		(property "Reference" "R6"
-			(at 118.11 57.7148 0)
+		(property "Reference" "F2"
+			(at 101.475 69.85 0)
 			(show_name no)
 			(do_not_autoplace no)
@@
 		)
 		(property "Value" "PTA6043-2015CPB103"
-			(at 118.11 60.2548 0)
+			(at 101.475 72.39 0)
 			(show_name no)
 			(do_not_autoplace no)
@@
 			(project "board"
 				(path "/a701f4fd-d5c8-4ab0-b464-3edf07ec58ed/58fefd48-2eee-4fcb-b0ad-9a73a5e36ec8"
-					(reference "R6")
+					(reference "F2")
 					(unit 1)
 				)
@@
 		(dnp no)
 		(fields_autoplaced yes)
-		(property "Reference" "SW16"
+		(property "Reference" "EN6"
 			(at 275.59 111.0548 0)
 			(show_name no)
@@
 			(project "board"
 				(path "/a701f4fd-d5c8-4ab0-b464-3edf07ec58ed/58fefd48-2eee-4fcb-b0ad-9a73a5e36ec8"
-					(reference "SW16")
+					(reference "EN6")
 					(unit 1)
 				)
@@
 		(dnp no)
 		(fields_autoplaced yes)
-		(property "Reference" "SW15"
+		(property "Reference" "EN5"
 			(at 242.57 110.4198 0)
 			(show_name no)
@@
 			(project "board"
 				(path "/a701f4fd-d5c8-4ab0-b464-3edf07ec58ed/58fefd48-2eee-4fcb-b0ad-9a73a5e36ec8"
-					(reference "SW15")
+					(reference "EN5")
 					(unit 1)
 				)
@@
 		(dnp no)
 		(fields_autoplaced yes)
-		(property "Reference" "R5"
-			(at 118.11 41.2048 0)
+		(property "Reference" "F1"
+			(at 101.475 53.34 0)
 			(show_name no)
 			(do_not_autoplace no)
@@
 		)
 		(property "Value" "PTA6043-2015CPB103"
-			(at 118.11 43.7448 0)
+			(at 101.475 55.88 0)
 			(show_name no)
 			(do_not_autoplace no)
@@
 			(project "board"
 				(path "/a701f4fd-d5c8-4ab0-b464-3edf07ec58ed/58fefd48-2eee-4fcb-b0ad-9a73a5e36ec8"
-					(reference "R5")
+					(reference "F1")
 					(unit 1)
 				)
@@
 		(dnp no)
 		(fields_autoplaced yes)
-		(property "Reference" "SW6"
+		(property "Reference" "M3"
 			(at 110.49 161.29 0)
 			(show_name no)
@@
 			(project "board"
 				(path "/a701f4fd-d5c8-4ab0-b464-3edf07ec58ed/58fefd48-2eee-4fcb-b0ad-9a73a5e36ec8"
-					(reference "SW6")
+					(reference "M3")
 					(unit 1)
 				)

Commit message: wiring and wiring
wiring and wiring
Parts:
- M1, M2, M3, M4, M5, M6, M7, M8: footprint easyeda_imports:KEY-TH_CPG151101D21X -> easyeda_imports:KEY-TH_CPG135001D0X
Other:
- moved on the sheet: M1, M2, M3, M4
