File: Hardware/board/led.kicad_sch (KiCad schematic)
At the start: 42 parts, among them U10 WS2812B, U11 WS2812B, U12 WS2812B, U13 WS2812B, U14 WS2812B, U15 WS2812B, U16 WS2812B, U17 WS2812B, U18 WS2812B, U19 WS2812B, U20 WS2812B, U21 WS2812B, U22 WS2812B, U23 WS2812B, U24 WS2812B, U25 WS2812B, U26 WS2812B, U27 WS2812B, U28 WS2812B, U29 WS2812B, U30 WS2812B, U31 WS2812B, U32 WS2812B, U33 WS2812B, U34 WS2812B, U35 WS2812B, U36 WS2812B, U37 WS2812B, U38 WS2812B, U39 WS2812B, U40 WS2812B, U41 WS2812B, U42 WS2812B, U43 WS2812B, U44 WS2812B, U45 WS2812B, U46 WS2812B, U47 WS2812B, U6 WS2812B, U7 WS2812B, U8 WS2812B, U9 WS2812B

Commit message: desigin designing
dsa
Parts:
- renumbered U7 to U10, U15 to U12, U19 to U13, U22 to U14, U8 to U15, U12 to U16, U16 to U17, U20 to U18, U41 to U19, U9 to U20, U13 to U21, U17 to U22, U21 to U23, U42 to U24, U43 to U25, U44 to U26, U45 to U27, U46 to U28, U26 to U29, U23 to U30, U29 to U31, U47 to U32, U27 to U33, U24 to U34, U30 to U35, U28 to U36, U25 to U37, U31 to U38, U32 to U39, U35 to U40, U38 to U41, U33 to U42, U36 to U43, U39 to U44, U34 to U45, U37 to U46, U40 to U47, U10 to U7, U14 to U8, U18 to U9
Connections:
- net 5V_LED renamed +5V_LED
- net E1_LED renamed LED_ENC1_DATA
- net E2_LED renamed LED_ENC2_DATA
- net E3_LED renamed LED_ENC3_DATA
- net E4_LED renamed LED_ENC4_DATA
- net E5_LED renamed LED_ENC5_DATA
- net F1_LED renamed LED_FADER1_DATA
- net F2_LED renamed LED_FADER2_DATA
- net F3_LED renamed LED_FADER3_DATA
- net F4_LED renamed LED_FADER4_DATA
- net M_LED renamed LED_KEYS_DATA

Commit message: i am cooked
Parts:
- removed U10, U11, U12, U13, U14, U15, U16, U17, U18, U19, U20, U21, U22, U23, U24, U25, U26, U27, U28, U29, U30, U31, U32, U33, U34, U35, U36, U37, U38, U39, U40, U41, U42, U43, U44, U45, U46, U47, U6, U7, U8, U9: WS2812B, easyeda_imports:LED-SMD_4P-L4.0-W1.7-R, symbol easyeda_imports:WS2812B-4020-G1
- added C22, C23, C24, C25, C26, C27, C28, C29, C30, C31, C32, C33, C34, C35, C36, C37, C38, C39, C40, C41, C42, C43, C44, C45, C46, C47, C48, C49, C50, C51, C52, C53, C54, C55, C56, C57, C58, C59, C60, C61, C62, C63: 100nF, PCM_fab:C_0603, symbol PCM_fab:C_0603
- added L1, L10, L11, L12, L13, L14, L15, L16, L17, L18, L19, L2, L20, L21, L22, L23, L24, L25, L26, L27, L28, L29, L3, L30, L31, L32, L33, L34, L35, L36, L37, L38, L39, L4, L40, L41, L42, L5, L6, L7, L8, L9: WS2812B, easyeda_imports:LED-SMD_4P-L2.0-W2.0-TL_WS2812B-2020, symbol easyeda_imports:WS2812B-2020
Connections:
- net +5V_LED: now also C22.1, C23.1, C24.1, C25.1, C26.1, C27.1, C28.1, C29.1, C30.1, C31.1, C32.1, C33.1, C34.1, C35.1, C36.1, C37.1, C38.1, C39.1, C40.1, C41.1, C42.1, C43.1, C44.1, C45.1, C46.1, C47.1, C48.1, C49.1, C50.1, C51.1, C52.1, C53.1, C54.1, C55.1, C56.1, C57.1, C58.1, C59.1, C60.1, C61.1, C62.1, C63.1, L1.4 (VDD), L10.4 (VDD), L11.4 (VDD), L12.4 (VDD), L13.4 (VDD), L14.4 (VDD), L15.4 (VDD), L16.4 (VDD), L17.4 (VDD), L18.4 (VDD), L19.4 (VDD), L2.4 (VDD), L20.4 (VDD), L21.4 (VDD), L22.4 (VDD), L23.4 (VDD), L24.4 (VDD), L25.4 (VDD), L26.4 (VDD), L27.4 (VDD), L28.4 (VDD), L29.4 (VDD), L3.4 (VDD), L30.4 (VDD), L31.4 (VDD), L32.4 (VDD), L33.4 (VDD), L34.4 (VDD), L35.4 (VDD), L36.4 (VDD), L37.4 (VDD), L38.4 (VDD), L39.4 (VDD), L4.4 (VDD), L40.4 (VDD), L41.4 (VDD), L42.4 (VDD), L5.4 (VDD), L6.4 (VDD), L7.4 (VDD), L8.4 (VDD), L9.4 (VDD)
- net GND: now also C22.2, C23.2, C24.2, C25.2, C26.2, C27.2, C28.2, C29.2, C30.2, C31.2, C32.2, C33.2, C34.2, C35.2, C36.2, C37.2, C38.2, C39.2, C40.2, C41.2, C42.2, C43.2, C44.2, C45.2, C46.2, C47.2, C48.2, C49.2, C50.2, C51.2, C52.2, C53.2, C54.2, C55.2, C56.2, C57.2, C58.2, C59.2, C60.2, C61.2, C62.2, C63.2, L1.2 (GND), L10.2 (GND), L11.2 (GND), L12.2 (GND), L13.2 (GND), L14.2 (GND), L15.2 (GND), L16.2 (GND), L17.2 (GND), L18.2 (GND), L19.2 (GND), L2.2 (GND), L20.2 (GND), L21.2 (GND), L22.2 (GND), L23.2 (GND), L24.2 (GND), L25.2 (GND), L26.2 (GND), L27.2 (GND), L28.2 (GND), L29.2 (GND), L3.2 (GND), L30.2 (GND), L31.2 (GND), L32.2 (GND), L33.2 (GND), L34.2 (GND), L35.2 (GND), L36.2 (GND), L37.2 (GND), L38.2 (GND), L39.2 (GND), L4.2 (GND), L40.2 (GND), L41.2 (GND), L42.2 (GND), L5.2 (GND), L6.2 (GND), L7.2 (GND), L8.2 (GND), L9.2 (GND)
- net LED_ENC1_DATA: now also L18.3 (DIN)
- net LED_ENC2_DATA: now also L17.3 (DIN)
- net LED_ENC3_DATA: now also L19.3 (DIN)
- net LED_ENC4_DATA: now also L32.3 (DIN)
- net LED_ENC5_DATA: now also L33.3 (DIN)
- net LED_FADER1_DATA: now also L1.3 (DIN)
- net LED_FADER2_DATA: now also L2.3 (DIN)
- net LED_FADER3_DATA: now also L3.3 (DIN)
- net LED_FADER4_DATA: now also L4.3 (DIN)
- net LED_KEYS_DATA: now also L20.3 (DIN)
- new net: L12.3 (DIN), L8.1 (DOUT)
- new net: L4.1 (DOUT), L8.3 (DIN)
- new net: L38.1 (DOUT), L42.3 (DIN)
- new net: L34.1 (DOUT), L38.3 (DIN)
- new net: L17.1 (DOUT), L21.3 (DIN)
- new net: L35.1 (DOUT), L39.3 (DIN)
- new net: L10.1 (DOUT), L14.3 (DIN)
- new net: L10.3 (DIN), L6.1 (DOUT)
- new net: L36.1 (DOUT), L40.3 (DIN)
- new net: L11.1 (DOUT), L15.3 (DIN)
- new net: L11.3 (DIN), L7.1 (DOUT)
- new net: L23.1 (DOUT), L27.3 (DIN)
- new net: L19.1 (DOUT), L23.3 (DIN)
- new net: L32.1 (DOUT), L36.3 (DIN)
- new net: L31.1 (DOUT), L35.3 (DIN)
- new net: L21.1 (DOUT), L25.3 (DIN)
- new net: L24.1 (DOUT), L28.3 (DIN)
- new net: L20.1 (DOUT), L24.3 (DIN)
- new net: L30.1 (DOUT), L34.3 (DIN)
- new net: L1.1 (DOUT), L5.3 (DIN)
- new net: L12.1 (DOUT), L16.3 (DIN)
- new net: L22.1 (DOUT), L26.3 (DIN)
- new net: L5.1 (DOUT), L9.3 (DIN)
- new net: L2.1 (DOUT), L6.3 (DIN)
- new net: L18.1 (DOUT), L22.3 (DIN)
- new net: L29.1 (DOUT), L30.3 (DIN)
- new net: L13.3 (DIN), L9.1 (DOUT)
- new net: L37.1 (DOUT), L41.3 (DIN)
- new net: L33.1 (DOUT), L37.3 (DIN)
- new net: L28.1 (DOUT), L29.3 (DIN)
- new net: L3.1 (DOUT), L7.3 (DIN)
- new net LED_ENC6_DATA: L31.3 (DIN)

Commit message: wiring and wiring
wiring and wiring
Parts:
- removed C41, C42, C43, C44, C45, C46, C50, C51, C52, C53, C54, C55: 100nF, PCM_fab:C_0603, symbol PCM_fab:C_0603
- removed L21, L22, L23, L25, L26, L27, L35, L36, L37, L39, L40, L41: WS2812B, easyeda_imports:LED-SMD_4P-L2.0-W2.0-TL_WS2812B-2020, symbol easyeda_imports:WS2812B-2020
