File: Hardware/board/mcu.kicad_sch (KiCad schematic)
At the start: 17 parts, among them SW1 SKRPACE010, U3 STM32F407VETx, X1 CSTNE8M00G550000R0

Commit message: hahahaahhahaha
Connections:
- net E4-S: now reaches U3.1 (PE2)
- net K1: now reaches U3.15 (PC0)
- net K2: now reaches U3.16 (PC1)
- net K3: now reaches U3.17 (PC2)
- net K4: now reaches U3.18 (PC3)
- net E5-A: now reaches U3.2 (PE3)
- net E6_LED: now reaches U3.29 (PA4)
- net E5-B: now reaches U3.3 (PE4)
- net K5: now reaches U3.33 (PC4)
- net E1-A: now reaches U3.35 (PB0)
- net E1-B: now reaches U3.36 (PB1)
- net E1-S: now reaches U3.37 (PB2)
- net E5-S: now reaches U3.4 (PE5)
- net F1_LED: now reaches U3.47 (PB10)
- net F2_LED: now reaches U3.48 (PB11)
- net F3_LED: now reaches U3.51 (PB12)
- net F4_LED: now reaches U3.52 (PB13)
- net E4_LED: now reaches U3.59 (PD12)
- net E5_LED: now reaches U3.60 (PD13)
- net K6: now reaches U3.63 (PC6)
- net K7: now reaches U3.64 (PC7)
- net E6-A: now reaches U3.65 (PC8)
- net E6-B: now reaches U3.66 (PC9)
- net M_LED: now reaches U3.67 (PA8)
- net E6-S: now reaches U3.78 (PC10)
- net K8: now reaches U3.79 (PC11)
- net E1_LED: now reaches U3.83 (PD2)
- net E2_LED: now reaches U3.84 (PD3)
- net E3_LED: now reaches U3.87 (PD6)
- net E2-A: now reaches U3.90 (PB4)
- net E2-B: now reaches U3.91 (PB5)
- net E2-S: now reaches U3.92 (PB6)
- net E3-A: now reaches U3.93 (PB7)
- net E3-B: now reaches U3.95 (PB8)
- net E3-S: now reaches U3.96 (PB9)
- net E4-A: now reaches U3.97 (PE0)
- net E4-B: now reaches U3.98 (PE1)

Commit message: desigin designing
dsa
Parts:
- renumbered C6 to C10, C15 to C11, C7 to C12, C8 to C13, C9 to C14, C10 to C15, C11 to C16, C12 to C17, C13 to C18, C16 to C6, C17 to C7, C5 to C8, C14 to C9
Connections:
- net 3.3V_MCU renamed +3.3V_DIGITAL
- net D+ renamed USB_D+
- net D- renamed USB_D-
- net D0 renamed FSMC_D0
- net D1 renamed FSMC_D1
- net D10 renamed FSMC_D10
- net D11 renamed FSMC_D11
- net D12 renamed FSMC_D12
- net D13 renamed FSMC_D13
- net D14 renamed FSMC_D14
- net D15 renamed FSMC_D15
- net D2 renamed FSMC_D2
- net D3 renamed FSMC_D3
- net D4 renamed FSMC_D4
- net D5 renamed FSMC_D5
- net D6 renamed FSMC_D6
- net D7 renamed FSMC_D7
- net D8 renamed FSMC_D8
- net D9 renamed FSMC_D9
- net E1-A renamed ENC1_A
- net E1-B renamed ENC1_B
- net E1-S renamed ENC1_SW
- net E1_LED renamed LED_ENC1_DATA
- net E2-A renamed ENC2_A
- net E2-B renamed ENC2_B
- net E2-S renamed ENC2_SW
- net E2_LED renamed LED_ENC2_DATA
- net E3-A renamed ENC3_A
- net E3-B renamed ENC3_B
- net E3-S renamed ENC3_SW
- net E3_LED renamed LED_ENC3_DATA
- net E4-A renamed ENC4_A
- net E4-B renamed ENC4_B
- net E4-S renamed ENC4_SW
- net E4_LED renamed LED_ENC4_DATA
- net E5-A renamed ENC5_A
- net E5-B renamed ENC5_B
- net E5-S renamed ENC5_SW
- net E5_LED renamed LED_ENC5_DATA
- net E6-A renamed ENC6_A
- net E6-B renamed ENC6_B
- net E6-S renamed ENC6_SW
- net E6_LED renamed LED_ENC6_DATA
- net F1_LED renamed LED_FADER1_DATA
- net F2_LED renamed LED_FADER2_DATA
- net F3_LED renamed LED_FADER3_DATA
- net F4_LED renamed LED_FADER4_DATA
- net K1 renamed SW_1
- net K2 renamed SW_2
- net K3 renamed SW_3
- net K4 renamed SW_4
- net K5 renamed SW_5
- net K6 renamed SW_6
- net K7 renamed SW_7
- net K8 renamed SW_8
- net LCS_CS renamed FSMC_NE1
- net LCS_RD renamed FSMC_NOE
- net LCS_RS renamed FSMC_A16
- net LCS_RST renamed LCD_RST
- net LCS_WR renamed FSMC_NWE
- net M_LED renamed LED_KEYS_DATA

Commit message: sdadsa
Parts:
- added R15: 10k, Resistor_SMD:R_0603_1608Metric, symbol PCM_Resistor_US_AKL:R_0603
- added SW16: SKRPACE010, easyeda_imports:KEY-SMD_4P-L4.2-W3.2-P2.20-LS4.6, symbol easyeda_imports:SKRPACE010
Connections:
- net +3.3V_DIGITAL: now also U3.21 (VREF+), R15.2
- net BOOT0: now also U3.94 (BOOT0)
- net GND: now also SW16.1, SW16.2
- net at U3.14 (NRST): now also R15.1, SW16.3, SW16.4

Commit message: i am cooked
Parts:
- renumbered C7 to C10, C8 to C11, C9 to C12, C10 to C13, C11 to C14, C12 to C15, C13 to C16, C14 to C17, C15 to C18, C16 to C19, C17 to C20, C18 to C21, C6 to C9, R15 to R3, R3 to R4, SW16 to SW1, SW1 to SW2
Connections:
- net FADER_1: now reaches U3.23 (PA0)
- net FADER_2: now reaches U3.24 (PA1)
- net FADER_4: now reaches U3.26 (PA3)
- net BACKLIGHT_PWM: now reaches U3.53 (PB14)

Commit message: wiring and wiring
wiring and wiring
Connections:
- net FADER_3: now also U3.25 (PA2)
Changed lines of the file:
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@@
 	(global_label "FADER_3"
 		(shape bidirectional)
-		(at 111.76 40.64 0)
+		(at 111.125 40.64 0)
 		(effects
 			(font
@@
 		)
 		(property "Intersheetrefs" "${INTERSHEET_REFS}"
-			(at 111.76 40.64 0)
+			(at 111.125 40.64 0)
 			(hide yes)
 			(show_name no)
