File: Hardware/board/power-usb.kicad_sch (KiCad schematic)
At the start: 11 parts, among them J1 USB_C_Receptacle_USB2.0_16P, J2 Barrel_Jack_PTH, U1 MIC5219-3.3YM5, U2 MIC5219-3.3YM5

Commit message: desigin designing
dsa
Parts:
- added C5: RVT1C102M1010, easyeda_imports:CAP-SMD_BD10.0-L10.3-W10.3-LS11.3-FD, symbol easyeda_imports:RVT1C102M1010
- renumbered C3 to C1, C1 to C2, C4 to C3, C2 to C4, U2 to U1, U1 to U2
Connections:
- net 3.3V_SYS is gone; now on net +3.3V_DIGITAL: C3.1, U1.5 (OUT)
- net 5V_SYS is gone; now on net +5V_SYS: C1.1, C2.1, D1.3 (K), U1.1 (IN), U1.3 (EN), U2.1 (IN), U2.3 (EN)
- net GND: now also C5.2
- net 12V renamed +12V
- net +12V: now also C5.1
- net 3.3V_MCU renamed +3.3V_DIGITAL
- net 5V_BUCK renamed +5V_SYS
- net D+ renamed USB_D+
- net D- renamed USB_D-
Changed lines of the file:
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@@
 		)
 	)
-	(label "5V_SYS"
+	(label "+12V"
+		(at 251.46 53.975 180)
+		(effects
+			(font
+				(size 1.27 1.27)
+			)
+			(justify right bottom)
+		)
+	)
+	(label "+5V_SYS"
 		(at 135.255 116.84 180)
 		(effects
@@
 		)
 	)
-	(label "5V_SYS"
+	(label "+5V_SYS"
 		(at 135.89 94.615 180)
 		(effects
@@
 		)
 	)
-	(label "12V"
+	(label "+12V"
 		(at 276.86 22.225 0)
 		(effects
@@
 		)
 	)
-	(label "D-"
+	(label "USB_D-"
 		(at 55.88 43.18 0)
 		(effects
@@
 		)
 	)
-	(label "D+"
+	(label "USB_D+"
 		(at 55.88 45.72 0)
 		(effects
@@
 		)
 	)
-	(label "5V_BUCK"
+	(label "+5V_SYS"
 		(at 154.305 40.64 180)
 		(effects
@@
 		)
 	)
-	(label "3.3V_MCU"
+	(label "+3.3V_DIGITAL"
 		(at 186.055 95.885 0)
 		(effects
@@
 		)
 	)
-	(label "5V_SYS"
+	(label "+5V_SYS"
 		(at 168.275 38.1 0)
 		(effects
@@
 		)
 	)
-	(label "3.3V_SYS"
+	(label "+3.3V_DIGITAL"
 		(at 185.42 118.11 0)
 		(effects
@@
 		(dnp no)
 		(fields_autoplaced yes)
-		(property "Reference" "U2"
+		(property "Reference" "U1"
 			(at 161.29 109.855 0)
 			(show_name no)
@@
 			(project "board"
 				(path "/a701f4fd-d5c8-4ab0-b464-3edf07ec58ed/3ef6c159-c183-4515-9efb-03480defbf53"
-					(reference "U2")
+					(reference "U1")
 					(unit 1)
 				)
@@
 		(dnp no)
 		(fields_autoplaced yes)
-		(property "Reference" "#PWR03"
+		(property "Reference" "#PWR010"
 			(at 283.21 27.305 0)
 			(hide yes)
@@
 			(project "board"
 				(path "/a701f4fd-d5c8-4ab0-b464-3edf07ec58ed/3ef6c159-c183-4515-9efb-03480defbf53"
-					(reference "#PWR03")
+					(reference "#PWR010")
 					(unit 1)
 				)
@@
 	(symbol
 		(lib_id "PCM_SparkFun-PowerSymbol:GND")
-		(at 177.165 125.73 0)
+		(at 259.08 53.975 90)
 		(unit 1)
 		(body_style 1)
@@
 		(fields_autoplaced yes)
 		(property "Reference" "#PWR09"
+			(at 265.43 53.975 0)
+			(hide yes)
+			(show_name no)
+			(do_not_autoplace no)
+			(effects
+				(font
+					(size 1.27 1.27)
+				)
+			)
+		)
+		(property "Value" "GND"
+			(at 262.89 53.975 0)
+			(show_name no)
+			(do_not_autoplace yes)
+			(effects
+				(font
+					(size 1.27 1.27)
+				)
+			)
+		)
+		(property "Footprint" ""
+			(at 259.08 53.975 0)
+			(hide yes)
+			(show_name no)
+			(do_not_autoplace no)
+			(effects
+				(font
+					(size 1.27 1.27)
+				)
+			)
+		)
+		(property "Datasheet" ""
+			(at 259.08 53.975 0)
+			(hide yes)
+			(show_name no)
+			(do_not_autoplace no)
+			(effects
+				(font
+					(size 1.27 1.27)
+				)
+			)
+		)
+		(property "Description" "Power symbol creates a global label with name \"GND\" , ground"
+			(at 267.97 53.975 0)
+			(hide yes)
+			(show_name no)
+			(do_not_autoplace no)
+			(effects
+				(font
+					(size 1.27 1.27)
+				)
+			)
+		)
+		(pin "1"
+		)
+		(instances
+			(project "board"
+				(path "/a701f4fd-d5c8-4ab0-b464-3edf07ec58ed/3ef6c159-c183-4515-9efb-03480defbf53"
+					(reference "#PWR09")
+					(unit 1)
+				)
+			)
+		)
+	)
+	(symbol
+		(lib_id "PCM_SparkFun-PowerSymbol:GND")
+		(at 177.165 125.73 0)
+		(unit 1)
+		(body_style 1)
+		(exclude_from_sim no)
+		(in_bom yes)
+		(on_board yes)
+		(in_pos_files yes)
+		(dnp no)
+		(fields_autoplaced yes)
+		(property "Reference" "#PWR07"
 			(at 177.165 132.08 0)
 			(hide yes)
@@
 			(project "board"
 				(path "/a701f4fd-d5c8-4ab0-b464-3edf07ec58ed/3ef6c159-c183-4515-9efb-03480defbf53"
-					(reference "#PWR09")
+					(reference "#PWR07")
 					(unit 1)
 				)
@@
 		(dnp no)
 		(fields_autoplaced yes)
-		(property "Reference" "#PWR02"
+		(property "Reference" "#PWR01"
 			(at 22.86 67.945 0)
 			(hide yes)
@@
 			(project "board"
 				(path "/a701f4fd-d5c8-4ab0-b464-3edf07ec58ed/3ef6c159-c183-4515-9efb-03480defbf53"
-					(reference "#PWR02")
+					(reference "#PWR01")
 					(unit 1)
 				)
@@
 		(in_pos_files yes)
 		(dnp no)
-		(property "Reference" "C1"
+		(property "Reference" "C2"
 			(at 142.24 97.155 0)
 			(show_name no)
@@
 			(project "board"
 				(path "/a701f4fd-d5c8-4ab0-b464-3edf07ec58ed/3ef6c159-c183-4515-9efb-03480defbf53"
-					(reference "C1")
+					(reference "C2")
 					(unit 1)
 				)
@@
 		(in_pos_files yes)
 		(dnp no)
-		(property "Reference" "C3"
+		(property "Reference" "C1"
 			(at 141.605 119.38 0)
 			(show_name no)
@@
 			(project "board"
 				(path "/a701f4fd-d5c8-4ab0-b464-3edf07ec58ed/3ef6c159-c183-4515-9efb-03480defbf53"
-					(reference "C3")
+					(reference "C1")
 					(unit 1)
 				)
@@
 		(dnp no)
 		(fields_autoplaced yes)
-		(property "Reference" "U1"
+		(property "Reference" "U2"
 			(at 161.925 87.63 0)
 			(show_name no)
@@
 			(project "board"
 				(path "/a701f4fd-d5c8-4ab0-b464-3edf07ec58ed/3ef6c159-c183-4515-9efb-03480defbf53"
-					(reference "U1")
+					(reference "U2")
 					(unit 1)
 				)
@@
 		(in_pos_files yes)
 		(dnp no)
-		(property "Reference" "C4"
+		(property "Reference" "C3"
 			(at 179.705 120.65 0)
 			(show_name no)
@@
 			(project "board"
 				(path "/a701f4fd-d5c8-4ab0-b464-3edf07ec58ed/3ef6c159-c183-4515-9efb-03480defbf53"
-					(reference "C4")
+					(reference "C3")
 					(unit 1)
 				)
@@
 		(in_pos_files yes)
 		(dnp no)
-		(property "Reference" "C2"
+		(property "Reference" "C4"
 			(at 180.34 98.425 0)
 			(show_name no)
@@
 			(project "board"
 				(path "/a701f4fd-d5c8-4ab0-b464-3edf07ec58ed/3ef6c159-c183-4515-9efb-03480defbf53"
-					(reference "C2")
+					(reference "C4")
 					(unit 1)
 				)
@@
 		(dnp no)
 		(fields_autoplaced yes)
-		(property "Reference" "#PWR01"
+		(property "Reference" "#PWR02"
 			(at 75.565 21.59 0)
 			(hide yes)
@@
 			(project "board"
 				(path "/a701f4fd-d5c8-4ab0-b464-3edf07ec58ed/3ef6c159-c183-4515-9efb-03480defbf53"
-					(reference "#PWR01")
+					(reference "#PWR02")
 					(unit 1)
 				)
@@
 		(dnp no)
 		(fields_autoplaced yes)
-		(property "Reference" "#PWR05"
+		(property "Reference" "#PWR04"
 			(at 139.7 108.585 0)
 			(hide yes)
@@
 			(project "board"
 				(path "/a701f4fd-d5c8-4ab0-b464-3edf07ec58ed/3ef6c159-c183-4515-9efb-03480defbf53"
-					(reference "#PWR05")
+					(reference "#PWR04")
 					(unit 1)
 				)
@@
 		(dnp no)
 		(fields_autoplaced yes)
-		(property "Reference" "#PWR08"
+		(property "Reference" "#PWR05"
 			(at 153.67 128.27 0)
 			(hide yes)
@@
 			(project "board"
 				(path "/a701f4fd-d5c8-4ab0-b464-3edf07ec58ed/3ef6c159-c183-4515-9efb-03480defbf53"
-					(reference "#PWR08")
+					(reference "#PWR05")
 					(unit 1)
 				)
@@
 		(dnp no)
 		(fields_autoplaced yes)
-		(property "Reference" "#PWR04"
+		(property "Reference" "#PWR06"
 			(at 154.305 106.045 0)
 			(hide yes)
@@
 			(project "board"
 				(path "/a701f4fd-d5c8-4ab0-b464-3edf07ec58ed/3ef6c159-c183-4515-9efb-03480defbf53"
-					(reference "#PWR04")
+					(reference "#PWR06")
+					(unit 1)
+				)
+			)
+		)
+	)
+	(symbol
+		(lib_id "easyeda_imports:RVT1C102M1010")
+		(at 255.27 53.975 0)
+		(unit 1)
+		(body_style 1)
+		(exclude_from_sim no)
+		(in_bom yes)
+		(on_board yes)
+		(in_pos_files yes)
+		(dnp no)
+		(fields_autoplaced yes)
+		(property "Reference" "C5"
+			(at 254.665 46.99 0)
+			(show_name no)
+			(do_not_autoplace no)
+			(effects
+				(font
+					(size 1.27 1.27)
+				)
+			)
+		)
+		(property "Value" "RVT1C102M1010"
+			(at 254.665 49.53 0)
+			(show_name no)
+			(do_not_autoplace no)
+			(effects
+				(font
+					(size 1.27 1.27)
+				)
+			)
+		)
+		(property "Footprint" "easyeda_imports:CAP-SMD_BD10.0-L10.3-W10.3-LS11.3-FD"
+			(at 255.27 61.595 0)
+			(hide yes)
+			(show_name no)
+			(do_not_autoplace no)
+			(effects
+				(font
+					(size 1.27 1.27)
+				)
+			)
+		)
+		(property "Datasheet" "https://lcsc.com/product-detail/Aluminum-Electrolytic-Capacitors-SMD_1000uF-16V-20_C72470.html"
+			(at 255.27 64.135 0)
+			(hide yes)
+			(show_name no)
+			(do_not_autoplace no)
+			(effects
+				(font
+					(size 1.27 1.27)
+				)
+			)
+		)
+		(property "Description" "1000uF 16V ±20%"
+			(at 255.27 53.975 0)
+			(hide yes)
+			(show_name no)
+			(do_not_autoplace no)
+			(effects
+				(font
+					(size 1.27 1.27)
+				)
+			)
+		)
+		(property "Manufacturer" "ROQANG(容强)"
+			(at 255.27 66.675 0)
+			(hide yes)
+			(show_name no)
+			(do_not_autoplace no)
+			(effects
+				(font
+					(size 1.27 1.27)
+				)
+			)
+		)
+		(property "MPN" "RVT1C102M1010"
+			(at 255.27 69.215 0)
+			(hide yes)
+			(show_name no)
+			(do_not_autoplace no)
+			(effects
+				(font
+					(size 1.27 1.27)
+				)
+			)
+		)
+		(property "LCSC Part" "C72470"
+			(at 255.27 71.755 0)
+			(hide yes)
+			(show_name no)
+			(do_not_autoplace no)
+			(effects
+				(font
+					(size 1.27 1.27)
+				)
+			)
+		)
+		(pin "2"
+		)
+		(pin "1"
+		)
+		(instances
+			(project "board"
+				(path "/a701f4fd-d5c8-4ab0-b464-3edf07ec58ed/3ef6c159-c183-4515-9efb-03480defbf53"
+					(reference "C5")
 					(unit 1)
 				)
@@
 		(dnp no)
 		(fields_autoplaced yes)
-		(property "Reference" "#PWR06"
+		(property "Reference" "#PWR08"
 			(at 177.8 109.855 0)
 			(hide yes)
@@
 			(project "board"
 				(path "/a701f4fd-d5c8-4ab0-b464-3edf07ec58ed/3ef6c159-c183-4515-9efb-03480defbf53"
-					(reference "#PWR06")
+					(reference "#PWR08")
 					(unit 1)
 				)
@@
 		(dnp no)
 		(fields_autoplaced yes)
-		(property "Reference" "#PWR07"
+		(property "Reference" "#PWR03"
 			(at 139.065 130.81 0)
 			(hide yes)
@@
 			(project "board"
 				(path "/a701f4fd-d5c8-4ab0-b464-3edf07ec58ed/3ef6c159-c183-4515-9efb-03480defbf53"
-					(reference "#PWR07")
-					(unit 1)
-				)
+					(reference "#PWR03")
+					(unit 1)
+				)

Commit message: sdadsa
Parts:
- added C40, C41: 1uF, PCM_fab:C_0603, symbol PCM_fab:C_0603
- added U51: MIC5219-3.3YM5, Package_TO_SOT_SMD:SOT-23-5, symbol Regulator_Linear:MIC5219-3.3YM5
Connections:
- net +5V_SYS: now also C40.1, U51.1 (IN), U51.3 (EN)
- net GND: now also C40.2, C41.2, U51.2 (GND)
- new net +3.3V_ANALOG: C41.1, U51.5 (OUT)

Commit message: i am cooked
Parts:
- removed C1, C3: 1uF, PCM_fab:C_0603, symbol PCM_fab:C_0603
- removed J2: Barrel_Jack_PTH, Connector_BarrelJack:BarrelJack_CUI_PJ-102AH_Horizontal, symbol PCM_SparkFun-Connector:Barrel_Jack_PTH
- removed U1: MIC5219-3.3YM5, Package_TO_SOT_SMD:SOT-23-5, symbol Regulator_Linear:MIC5219-3.3YM5
- added C5, C6, C7: RVT1C102M1010, easyeda_imports:CAP-SMD_BD10.0-L10.3-W10.3-LS11.3-FD, symbol easyeda_imports:RVT1C102M1010
- added CN1: XT30PW-M, easyeda_imports:CONN-TH_XT30PW-M, symbol easyeda_imports:XT30PW-M
- renumbered C40 to C1, C41 to C3, C5 to C8, U51 to U1
Connections:
- net +12V: now also C5.1, C6.1, C7.1, CN1.2 (+)
- net GND: now also C5.2, C6.2, C7.2, CN1.1 (-)

Commit message: i hate it
Other:
- moved on the sheet: C5, C6, C7, C8
Changed lines of the file:
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@@
 	(global_label "+12V"
 		(shape bidirectional)
-		(at 251.46 53.975 180)
+		(at 248.92 48.895 180)
 		(effects
 			(font
@@
 		)
 		(property "Intersheetrefs" "${INTERSHEET_REFS}"
-			(at 251.46 53.975 0)
+			(at 248.92 48.895 0)
 			(hide yes)
 			(show_name no)
@@
 	(global_label "+12V"
 		(shape bidirectional)
-		(at 250.825 63.5 180)
+		(at 248.92 59.69 180)
 		(effects
 			(font
@@
 		)
 		(property "Intersheetrefs" "${INTERSHEET_REFS}"
-			(at 250.825 63.5 0)
+			(at 248.92 59.69 0)
 			(hide yes)
 			(show_name no)
@@
 	(global_label "+12V"
 		(shape bidirectional)
-		(at 250.19 73.025 180)
+		(at 249.555 69.85 180)
 		(effects
 			(font
@@
 		)
 		(property "Intersheetrefs" "${INTERSHEET_REFS}"
-			(at 250.19 73.025 0)
+			(at 249.555 69.85 0)
 			(hide yes)
 			(show_name no)
@@
 	(global_label "+12V"
 		(shape bidirectional)
-		(at 249.555 81.915 180)
+		(at 248.92 80.645 180)
 		(effects
 			(font
@@
 		)
 		(property "Intersheetrefs" "${INTERSHEET_REFS}"
-			(at 249.555 81.915 0)
+			(at 248.92 80.645 0)
 			(hide yes)
 			(show_name no)
@@
 	(symbol
 		(lib_id "easyeda_imports:RVT1C102M1010")
-		(at 254 73.025 0)
+		(at 253.365 69.85 0)
 		(unit 1)
 		(body_style 1)
@@
 		(fields_autoplaced yes)
 		(property "Reference" "C6"
-			(at 253.395 66.04 0)
+			(at 252.76 62.865 0)
 			(show_name no)
 			(do_not_autoplace no)
@@
 		)
 		(property "Value" "RVT1C102M1010"
-			(at 253.395 68.58 0)
+			(at 252.76 65.405 0)
 			(show_name no)
 			(do_not_autoplace no)
@@
 		)
 		(property "Footprint" "easyeda_imports:CAP-SMD_BD10.0-L10.3-W10.3-LS11.3-FD"
-			(at 254 80.645 0)
+			(at 253.365 77.47 0)
 			(hide yes)
 			(show_name no)
@@
 		)
 		(property "Datasheet" "https://lcsc.com/product-detail/Aluminum-Electrolytic-Capacitors-SMD_1000uF-16V-20_C72470.html"
-			(at 254 83.185 0)
+			(at 253.365 80.01 0)
 			(hide yes)
 			(show_name no)
@@
 		)
 		(property "Description" "1000uF 16V ±20%"
-			(at 254 73.025 0)
+			(at 253.365 69.85 0)
 			(hide yes)
 			(show_name no)
@@
 		)
 		(property "Manufacturer" "ROQANG(容强)"
-			(at 254 85.725 0)
+			(at 253.365 82.55 0)
 			(hide yes)
 			(show_name no)
@@
 		)
 		(property "MPN" "RVT1C102M1010"
-			(at 254 88.265 0)
+			(at 253.365 85.09 0)
 			(hide yes)
 			(show_name no)
@@
 		)
 		(property "LCSC Part" "C72470"
-			(at 254 90.805 0)
+			(at 253.365 87.63 0)
 			(hide yes)
 			(show_name no)
@@
 	(symbol
 		(lib_id "PCM_SparkFun-PowerSymbol:GND")
-		(at 259.08 53.975 90)
+		(at 256.54 48.895 90)
 		(unit 1)
 		(body_style 1)
@@
 		(fields_autoplaced yes)
 		(property "Reference" "#PWR013"
-			(at 265.43 53.975 0)
+			(at 262.89 48.895 0)
 			(hide yes)
 			(show_name no)
@@
 		)
 		(property "Value" "GND"
-			(at 262.89 53.975 0)
+			(at 260.35 48.895 0)
 			(show_name no)
 			(do_not_autoplace yes)
@@
 		)
 		(property "Footprint" ""
-			(at 259.08 53.975 0)
+			(at 256.54 48.895 0)
 			(hide yes)
 			(show_name no)
@@
 		)
 		(property "Datasheet" ""
-			(at 259.08 53.975 0)
+			(at 256.54 48.895 0)
 			(hide yes)
 			(show_name no)
@@
 		)
 		(property "Description" "Power symbol creates a global label with name \"GND\" , ground"
-			(at 267.97 53.975 0)
+			(at 265.43 48.895 0)
 			(hide yes)
 			(show_name no)
@@
 	(symbol
 		(lib_id "PCM_SparkFun-PowerSymbol:GND")
-		(at 257.81 73.025 90)
+		(at 257.175 69.85 90)
 		(unit 1)
 		(body_style 1)
@@
 		(fields_autoplaced yes)
 		(property "Reference" "#PWR011"
-			(at 264.16 73.025 0)
+			(at 263.525 69.85 0)
 			(hide yes)
 			(show_name no)
@@
 		)
 		(property "Value" "GND"
-			(at 261.62 73.025 0)
+			(at 260.985 69.85 0)
 			(show_name no)
 			(do_not_autoplace yes)
@@
 		)
 		(property "Footprint" ""
-			(at 257.81 73.025 0)
+			(at 257.175 69.85 0)
 			(hide yes)
 			(show_name no)
@@
 		)
 		(property "Datasheet" ""
-			(at 257.81 73.025 0)
+			(at 257.175 69.85 0)
 			(hide yes)
 			(show_name no)
@@
 		)
 		(property "Description" "Power symbol creates a global label with name \"GND\" , ground"
-			(at 266.7 73.025 0)
+			(at 266.065 69.85 0)
 			(hide yes)
 			(show_name no)
@@
 	(symbol
 		(lib_id "PCM_SparkFun-PowerSymbol:GND")
-		(at 257.175 81.915 90)
+		(at 256.54 80.645 90)
 		(unit 1)
 		(body_style 1)
@@
 		(fields_autoplaced yes)
 		(property "Reference" "#PWR010"
-			(at 263.525 81.915 0)
+			(at 262.89 80.645 0)
 			(hide yes)
 			(show_name no)
@@
 		)
 		(property "Value" "GND"
-			(at 260.985 81.915 0)
+			(at 260.35 80.645 0)
 			(show_name no)
 			(do_not_autoplace yes)
@@
 		)
 		(property "Footprint" ""
-			(at 257.175 81.915 0)
+			(at 256.54 80.645 0)
 			(hide yes)
 			(show_name no)
@@
 		)
 		(property "Datasheet" ""
-			(at 257.175 81.915 0)
+			(at 256.54 80.645 0)
 			(hide yes)
 			(show_name no)
@@
 		)
 		(property "Description" "Power symbol creates a global label with name \"GND\" , ground"
-			(at 266.065 81.915 0)
+			(at 265.43 80.645 0)
 			(hide yes)
 			(show_name no)
@@
 	(symbol
 		(lib_id "easyeda_imports:RVT1C102M1010")
-		(at 254.635 63.5 0)
+		(at 252.73 59.69 0)
 		(unit 1)
 		(body_style 1)
@@
 		(fields_autoplaced yes)
 		(property "Reference" "C7"
-			(at 254.03 56.515 0)
+			(at 252.125 52.705 0)
 			(show_name no)
 			(do_not_autoplace no)
@@
 		)
 		(property "Value" "RVT1C102M1010"
-			(at 254.03 59.055 0)
+			(at 252.125 55.245 0)
 			(show_name no)
 			(do_not_autoplace no)
@@
 		)
 		(property "Footprint" "easyeda_imports:CAP-SMD_BD10.0-L10.3-W10.3-LS11.3-FD"
-			(at 254.635 71.12 0)
+			(at 252.73 67.31 0)
 			(hide yes)
 			(show_name no)
@@
 		)
 		(property "Datasheet" "https://lcsc.com/product-detail/Aluminum-Electrolytic-Capacitors-SMD_1000uF-16V-20_C72470.html"
-			(at 254.635 73.66 0)
+			(at 252.73 69.85 0)
 			(hide yes)
 			(show_name no)
@@
 		)
 		(property "Description" "1000uF 16V ±20%"
-			(at 254.635 63.5 0)
+			(at 252.73 59.69 0)
 			(hide yes)
 			(show_name no)
@@
 		)
 		(property "Manufacturer" "ROQANG(容强)"
-			(at 254.635 76.2 0)
+			(at 252.73 72.39 0)
 			(hide yes)
 			(show_name no)
@@
 		)
 		(property "MPN" "RVT1C102M1010"
-			(at 254.635 78.74 0)
+			(at 252.73 74.93 0)
 			(hide yes)
 			(show_name no)
@@
 		)
 		(property "LCSC Part" "C72470"
-			(at 254.635 81.28 0)
+			(at 252.73 77.47 0)
 			(hide yes)
 			(show_name no)
@@
 	(symbol
 		(lib_id "PCM_SparkFun-PowerSymbol:GND")
-		(at 258.445 63.5 90)
+		(at 256.54 59.69 90)
 		(unit 1)
 		(body_style 1)
@@
 		(fields_autoplaced yes)
 		(property "Reference" "#PWR012"
-			(at 264.795 63.5 0)
+			(at 262.89 59.69 0)
 			(hide yes)
 			(show_name no)
@@
 		)
 		(property "Value" "GND"
-			(at 262.255 63.5 0)
+			(at 260.35 59.69 0)
 			(show_name no)
 			(do_not_autoplace yes)
@@
 		)
 		(property "Footprint" ""
-			(at 258.445 63.5 0)
+			(at 256.54 59.69 0)
 			(hide yes)
 			(show_name no)
@@
 		)
 		(property "Datasheet" ""
-			(at 258.445 63.5 0)
+			(at 256.54 59.69 0)
 			(hide yes)
 			(show_name no)
@@
 		)
 		(property "Description" "Power symbol creates a global label with name \"GND\" , ground"
-			(at 267.335 63.5 0)
+			(at 265.43 59.69 0)
 			(hide yes)
 			(show_name no)
@@
 	(symbol
 		(lib_id "easyeda_imports:RVT1C102M1010")
-		(at 255.27 53.975 0)
+		(at 252.73 48.895 0)
 		(unit 1)
 		(body_style 1)
@@
 		(fields_autoplaced yes)
 		(property "Reference" "C8"
-			(at 254.665 46.99 0)
+			(at 252.125 41.91 0)
 			(show_name no)
 			(do_not_autoplace no)
@@
 		)
 		(property "Value" "RVT1C102M1010"
-			(at 254.665 49.53 0)
+			(at 252.125 44.45 0)
 			(show_name no)
 			(do_not_autoplace no)
@@
 		)
 		(property "Footprint" "easyeda_imports:CAP-SMD_BD10.0-L10.3-W10.3-LS11.3-FD"
-			(at 255.27 61.595 0)
+			(at 252.73 56.515 0)
 			(hide yes)
 			(show_name no)
@@
 		)
 		(property "Datasheet" "https://lcsc.com/product-detail/Aluminum-Electrolytic-Capacitors-SMD_1000uF-16V-20_C72470.html"
-			(at 255.27 64.135 0)
+			(at 252.73 59.055 0)
 			(hide yes)
 			(show_name no)
@@
 		)
 		(property "Description" "1000uF 16V ±20%"
-			(at 255.27 53.975 0)
+			(at 252.73 48.895 0)
 			(hide yes)
 			(show_name no)
@@
 		)
 		(property "Manufacturer" "ROQANG(容强)"
-			(at 255.27 66.675 0)
+			(at 252.73 61.595 0)
 			(hide yes)
 			(show_name no)
@@
 		)
 		(property "MPN" "RVT1C102M1010"
-			(at 255.27 69.215 0)
+			(at 252.73 64.135 0)
 			(hide yes)
 			(show_name no)
@@
 		)
 		(property "LCSC Part" "C72470"
-			(at 255.27 71.755 0)
+			(at 252.73 66.675 0)
 			(hide yes)
 			(show_name no)
@@
 	(symbol
 		(lib_id "easyeda_imports:RVT1C102M1010")
-		(at 253.365 81.915 0)
+		(at 252.73 80.645 0)
 		(unit 1)
 		(body_style 1)
@@
 		(in_pos_files yes)
 		(dnp no)
-		(fields_autoplaced yes)
 		(property "Reference" "C5"
-			(at 252.76 74.93 0)
+			(at 252.73 73.66 0)
 			(show_name no)
 			(do_not_autoplace no)
@@
 		)
 		(property "Value" "RVT1C102M1010"
-			(at 252.76 77.47 0)
+			(at 252.125 76.2 0)
 			(show_name no)
 			(do_not_autoplace no)
@@
 		)
 		(property "Footprint" "easyeda_imports:CAP-SMD_BD10.0-L10.3-W10.3-LS11.3-FD"
-			(at 253.365 89.535 0)
+			(at 252.73 88.265 0)
 			(hide yes)
 			(show_name no)
@@
 		)
 		(property "Datasheet" "https://lcsc.com/product-detail/Aluminum-Electrolytic-Capacitors-SMD_1000uF-16V-20_C72470.html"
-			(at 253.365 92.075 0)
+			(at 252.73 90.805 0)
 			(hide yes)
 			(show_name no)
@@
 		)
 		(property "Description" "1000uF 16V ±20%"
-			(at 253.365 81.915 0)
+			(at 252.73 80.645 0)
 			(hide yes)
 			(show_name no)
@@
 		)
 		(property "Manufacturer" "ROQANG(容强)"
-			(at 253.365 94.615 0)
+			(at 252.73 93.345 0)
 			(hide yes)
 			(show_name no)
@@
 		)
 		(property "MPN" "RVT1C102M1010"
-			(at 253.365 97.155 0)
+			(at 252.73 95.885 0)
 			(hide yes)
 			(show_name no)
@@
 		)
 		(property "LCSC Part" "C72470"
-			(at 253.365 99.695 0)
-			(hide yes)
-			(show_name no)
+			(at 252.73 98.425 0)
+			(hide yes)
+			(show_name no)
