File: Hardware/board/power-usb.kicad_sch (KiCad schematic)
At the start: 15 parts, among them CN1 XT30PW-M, J1 USB_C_Receptacle_USB2.0_16P, U1 MIC5219-3.3YM5, U2 MIC5219-3.3YM5

Commit message: psuhing  and pushing
psuhing  and pushing
Parts:
- renumbered C8 to C5, C7 to C6, C5 to C7, C6 to C8
Changed lines of the file:
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@@
 		(dnp no)
 		(fields_autoplaced yes)
-		(property "Reference" "C6"
+		(property "Reference" "C8"
 			(at 252.76 62.865 0)
 			(show_name no)
@@
 			(project "board"
 				(path "/a701f4fd-d5c8-4ab0-b464-3edf07ec58ed/3ef6c159-c183-4515-9efb-03480defbf53"
-					(reference "C6")
+					(reference "C8")
 					(unit 1)
 				)
@@
 		(dnp no)
 		(fields_autoplaced yes)
-		(property "Reference" "#PWR013"
+		(property "Reference" "#PWR010"
 			(at 262.89 48.895 0)
 			(hide yes)
@@
 			(project "board"
 				(path "/a701f4fd-d5c8-4ab0-b464-3edf07ec58ed/3ef6c159-c183-4515-9efb-03480defbf53"
-					(reference "#PWR013")
+					(reference "#PWR010")
 					(unit 1)
 				)
@@
 		(dnp no)
 		(fields_autoplaced yes)
-		(property "Reference" "#PWR011"
+		(property "Reference" "#PWR013"
 			(at 263.525 69.85 0)
 			(hide yes)
@@
 			(project "board"
 				(path "/a701f4fd-d5c8-4ab0-b464-3edf07ec58ed/3ef6c159-c183-4515-9efb-03480defbf53"
-					(reference "#PWR011")
+					(reference "#PWR013")
 					(unit 1)
 				)
@@
 		(dnp no)
 		(fields_autoplaced yes)
-		(property "Reference" "#PWR010"
+		(property "Reference" "#PWR012"
 			(at 262.89 80.645 0)
 			(hide yes)
@@
 			(project "board"
 				(path "/a701f4fd-d5c8-4ab0-b464-3edf07ec58ed/3ef6c159-c183-4515-9efb-03480defbf53"
-					(reference "#PWR010")
+					(reference "#PWR012")
 					(unit 1)
 				)
@@
 		(dnp no)
 		(fields_autoplaced yes)
-		(property "Reference" "C7"
+		(property "Reference" "C6"
 			(at 252.125 52.705 0)
 			(show_name no)
@@
 			(project "board"
 				(path "/a701f4fd-d5c8-4ab0-b464-3edf07ec58ed/3ef6c159-c183-4515-9efb-03480defbf53"
-					(reference "C7")
+					(reference "C6")
 					(unit 1)
 				)
@@
 		(dnp no)
 		(fields_autoplaced yes)
-		(property "Reference" "#PWR012"
+		(property "Reference" "#PWR011"
 			(at 262.89 59.69 0)
 			(hide yes)
@@
 			(project "board"
 				(path "/a701f4fd-d5c8-4ab0-b464-3edf07ec58ed/3ef6c159-c183-4515-9efb-03480defbf53"
-					(reference "#PWR012")
+					(reference "#PWR011")
 					(unit 1)
 				)
@@
 		(dnp no)
 		(fields_autoplaced yes)
-		(property "Reference" "C8"
+		(property "Reference" "C5"
 			(at 252.125 41.91 0)
 			(show_name no)
@@
 			(project "board"
 				(path "/a701f4fd-d5c8-4ab0-b464-3edf07ec58ed/3ef6c159-c183-4515-9efb-03480defbf53"
-					(reference "C8")
+					(reference "C5")
 					(unit 1)
 				)
@@
 		(in_pos_files yes)
 		(dnp no)
-		(property "Reference" "C5"
+		(property "Reference" "C7"
 			(at 252.73 73.66 0)
 			(show_name no)
@@
 			(project "board"
 				(path "/a701f4fd-d5c8-4ab0-b464-3edf07ec58ed/3ef6c159-c183-4515-9efb-03480defbf53"
-					(reference "C5")
-					(unit 1)
-				)
+					(reference "C7")
+					(unit 1)
+				)

Commit message: wiring and wiring
wiring and wiring
Parts:
- removed C6, C7: RVT1C102M1010, easyeda_imports:CAP-SMD_BD10.0-L10.3-W10.3-LS11.3-FD, symbol easyeda_imports:RVT1C102M1010
- removed D1: PMEG4005CT, PCM_Package_TO_SOT_SMD_AKL:SOT-23, symbol PCM_Diode_Schottky_AKL:PMEG4005CT
Connections:
- net 5V_USB is gone; now on net +5V_SYS: J1.A4 (VBUS), J1.A9 (VBUS), J1.B4 (VBUS), J1.B9 (VBUS)
